File: pcb/batta pinky cluster/batta.kicad_pcb (KiCad board)
At the start: 2 copper layers, 126.9 x 99.3 mm, 43 parts

Commit message: ney keebs
Parts:
- removed MCU1: , ProMicro
- removed S10, S12, S14, S16, S18, S2, S20, S22, S24, S26, S28, S30, S32, S34, S4, S6, S8: , PG1350
- ?: moved to B.Cu
- S1, S11, S13, S15, S17, S19, S21, S23, S25, S27, S29, S3, S31, S33, S5, S7, S9: footprint PG1350 -> Alaa:key
- moved ? 116.1 mm to (38.6, -105.9)
- moved S1 34.0 mm to (38.6, -72.9)
- moved PAD1 22.6 mm to (151.9, -78.2)
- moved T1 19.0 mm to (157.3, -91.7)
- moved T2 19.0 mm to (157.3, -91.7)
- moved S33 5.96 mm to (148.3, -45.6), turned to -19 degrees
- moved B1 5.38 mm to (156.7, -60.7), turned to 90 degrees
- moved S31 5.31 mm to (128.6, -49.6), turned to -4 degrees
- moved S5 2.24 mm to (54.7, -83.4)
- moved S3 2.24 mm to (59.6, -67.1)
- moved S11 1.33 mm to (72.7, -105.0)
- moved S7 1.33 mm to (78.6, -71.5)
- moved S9 1.33 mm to (75.7, -88.2)
- moved REF** 1.25 mm to (104.1, -87.0)
- moved S13 0.68 mm to (96.4, -80.2)
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Connections:
- ? pad 1: (no net) -> RAW
- ? pad 10: (no net) -> P14
- ? pad 11: (no net) -> P16
- ? pad 12: (no net) -> P10
- ? pad 13: (no net) -> P9
- ? pad 14: (no net) -> P8
- ? pad 15: (no net) -> P7
- ? pad 16: (no net) -> P6
- ? pad 17: (no net) -> P5
- ? pad 18: (no net) -> P4
- ? pad 19: (no net) -> P3
- ? pad 2: (no net) -> GND
- ? pad 20: (no net) -> P2
- ? pad 21: (no net) -> GND
- ? pad 22: (no net) -> GND
- ? pad 23: (no net) -> P0
- ? pad 24: RAW -> P1
- ? pad 3: (no net) -> RST
- ? pad 4: (no net) -> VCC
- ? pad 5: (no net) -> P21
- ? pad 6: (no net) -> P20
- ? pad 7: (no net) -> P19
- ? pad 8: (no net) -> P18
- ? pad 9: (no net) -> P15
- PAD1 pad 2: Bminus -> GND
- S1 pad 1: P6 -> P14
- S11 pad 1: P0 -> P19
- S13 pad 1: P1 -> P4
- S15 pad 1: P18 -> P20
- S17 pad 1: P15 -> P21
- S19 pad 1: P14 -> P6
- S21 pad 1: P16 -> P2
- S23 pad 1: P10 -> P1
- S25 pad 1: P19 -> P7
- S27 pad 1: P20 -> P3
- S29 pad 1: P21 -> P0
- S3 pad 1: P5 -> P16
- S31 pad 1: P7 -> P9
- S5 pad 1: P4 -> P10
- S7 pad 1: P3 -> P5
- S9 pad 1: P2 -> P18
Routing:
- net RST: track 0.00 -> 191.9 mm
- net P9: track 0.00 -> 156.2 mm
- net P8: track 31.7 -> 181.8 mm
- net P7: track 31.7 -> 163.0 mm
- net RAW: track 12.4 -> 142.2 mm, vias 2 -> 1
- net P6: track 31.8 -> 146.7 mm
- net P3: track 31.6 -> 145.4 mm
- net P0: track 31.6 -> 142.4 mm
- net P2: track 31.6 -> 129.0 mm
- net P1: track 31.5 -> 126.2 mm
- net P4: track 31.8 -> 115.6 mm
- net P5: track 31.8 -> 101.4 mm
- net P20: track 31.2 -> 96.6 mm
- net P21: track 31.2 -> 85.5 mm
- net P16: track 31.5 -> 81.1 mm
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Other:
- board size 126.9 x 99.3 mm -> 133.4 x 90.7 mm
