File: boards/battoota_min/battoota_min.kicad_pcb (KiCad board)
At the start: 2 copper layers, 109.9 x 82.1 mm, 17 parts

Commit message: min versions routing
Parts:
- added B1: , kbd:ResetSW, F.Cu at (195.7, 77.8)
- added PAD1: , lib:bat, F.Cu at (205.0, 66.3)
- added T1, T2: , E73:SPDT_C128955, F.Cu at (195.0, 64.1)
- moved S10 4.10 mm to (261.1, 88.6)
- moved S11 4.10 mm to (261.1, 73.1)
- moved S12 4.10 mm to (277.6, 96.3)
- moved S13 4.10 mm to (277.6, 80.8)
- moved S9 4.10 mm to (261.1, 104.1)
- moved ? 1.31 mm to (269.3, 81.7)
- moved S1 1.00 mm to (207.3, 108.3)
- moved S2 1.00 mm to (202.7, 93.5)
- moved MCU1 0.89 mm to (212.1, 127.6)
Connections:
- S1 pad : (no net) -> P20
- S1 pad 1: GND -> P20
- S1 pad 2: P7 -> P20
- S10 pad : (no net) -> P8
- S10 pad 1: GND -> P8
- S10 pad 2: P16 -> GND
- S11 pad : (no net) -> P7
- S11 pad 1: GND -> P7
- S11 pad 2: P10 -> P7
- S12 pad 2: P19 -> P6
- S13 pad 1: GND -> P5
- S13 pad 2: P20 -> GND
- S14 pad : (no net) -> P4
- S14 pad 1: GND -> P4
- S14 pad 2: P8 -> P4
- S15 pad : (no net) -> P3
- S15 pad 1: GND -> P3
- S15 pad 2: P9 -> GND
- S2 pad : (no net) -> P21
- S2 pad 1: GND -> P21
- S2 pad 2: P6 -> P21
- S3 pad : (no net) -> P15
- S3 pad 1: GND -> P15
- S3 pad 2: P5 -> GND
- S4 pad : (no net) -> P18
- S4 pad 1: GND -> P18
- S4 pad 2: P4 -> P18
- S5 pad : (no net) -> P19
- S5 pad 2: P3 -> GND
- S6 pad : (no net) -> P10
- S6 pad 2: P2 -> GND
- S7 pad : (no net) -> P16
- S7 pad 2: P18 -> GND
- S8 pad : (no net) -> P14
- S8 pad 1: GND -> P14
- S8 pad 2: P15 -> GND
- S9 pad : (no net) -> P9
- S9 pad 1: GND -> P9
- S9 pad 2: P14 -> GND
Routing:
- net P5: track 31.4 -> 146.8 mm
- net RAW: track 0.00 -> 91.9 mm, vias 0 -> 2
- net P6: track 32.6 -> 112.0 mm
- net P3: track 33.2 -> 108.0 mm
- net P7: track 32.4 -> 106.9 mm
- net RST: track 0.00 -> 65.2 mm, vias 0 -> 1
- net P4: track 30.1 -> 93.0 mm
- net P9: track 32.1 -> 93.5 mm
- net P21: track 0.00 -> 60.4 mm
- net P14: track 31.8 -> 90.9 mm
- net P8: track 31.9 -> 90.2 mm
- net P19: track 32.3 -> 74.5 mm
- net BRAW: track 0.00 -> 41.8 mm
- net P16: track 31.8 -> 71.9 mm
- net P2: track 31.7 -> 0.00 mm
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Other:
- board size 109.9 x 82.1 mm -> 110.9 x 82.1 mm
