File: boards/Konafa/konafa.kicad_pcb (KiCad board)
At the start: 2 copper layers, 122.6 x 88.9 mm, 40 parts

Commit message: konafa cleanup
Parts:
- removed S10, S12, S14, S16, S18, S20, S22, S24 (x2), S28, S30, S32, S34, S4, S6, S8: , PG1350
- S11, S13, S15, S17, S19, S21, S23 (x2), S27, S29, S3, S31, S33, S5, S7, S9: footprint PG1350 -> Alaa:choc_hotswap_key
Connections:
- S11 pad : P3 -> (no net)
- S13 pad : P2 -> (no net)
- S23 pad : P21 -> (no net)
- S27 pad : P19 -> (no net)
- S29 pad : P20 -> (no net)
- S7 pad : P5 -> (no net)
- S9 pad : P4 -> (no net)
Routing:
- net Braw: track 57.1 -> 57.6 mm

Commit message: clean up all the boards
Routing:
- net GND: track 281.1 -> 7.75 mm
- added copper zone on F.Cu, net GND
- removed copper zone on F.Cu, net (none)
Changed lines of the file:
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@@
   (segment (start 47.655954 -88.184596) (end 48.856953 -86.983597) (width 0.25) (layer "B.Cu") (net 1))
   (segment (start 48.856953 -86.983597) (end 48.856953 -78.356283) (width 0.25) (layer "B.Cu") (net 1))
-  (segment (start 141.549822 -49.832832) (end 143.691642 -52.129654) (width 0.5) (layer "F.Cu") (net 2))
-  (segment (start 63.384822 -105.421809) (end 62.586645 -106.219986) (width 0.5) (layer "F.Cu") (net 2))
-  (segment (start 96.21751 -74.301308) (end 89.760656 -74.301308) (width 0.5) (layer "F.Cu") (net 2))
-  (segment (start 63.384822 -100.80225) (end 63.384822 -105.421809) (width 0.5) (layer "F.Cu") (net 2))
-  (segment (start 75.363653 -82.192969) (end 74.347654 -81.17697) (width 0.5) (layer "F.Cu") (net 2))
-  (segment (start 62.586645 -106.219986) (end 62.586645 -107.001157) (width 0.5) (layer "F.Cu") (net 2))
-  (segment (start 107.136087 -84.663616) (end 108.987449 -82.812254) (width 0.5) (layer "F.Cu") (net 2))
-  (segment (start 127.904087 -81.687254) (end 125.217087 -84.374254) (width 0.5) (layer "F.Cu") (net 2))
-  (segment (start 66.26837 -97.918702) (end 63.384822 -100.80225) (width 0.5) (layer "F.Cu") (net 2))
-  (segment (start 133.505791 -81.711491) (end 133.481554 -81.687254) (width 0.5) (layer "F.Cu") (net 2))
-  (segment (start 74.347654 -81.17697) (end 68.485407 -81.17697) (width 0.5) (layer "F.Cu") (net 2))
-  (segment (start 71.813295 -64.435238) (end 68.490683 -67.75785) (width 0.5) (layer "F.Cu") (net 2))
-  (segment (start 109.709791 -65.812254) (end 108.167264 -67.354781) (width 0.5) (layer "F.Cu") (net 2))
-  (segment (start 141.797987 -42.726297) (end 141.549822 -49.832832) (width 0.5) (layer "F.Cu") (net 2))
-  (segment (start 109.579975 -99.812254) (end 115.424791 -99.812254) (width 0.5) (layer "F.Cu") (net 2))
-  (segment (start 89.760656 -74.301308) (end 87.132946 -76.929018) (width 0.5) (layer "F.Cu") (net 2))
-  (segment (start 125.217087 -67.102254) (end 125.217087 -74.347787) (width 0.5) (layer "F.Cu") (net 2))
-  (segment (start 49.917361 -65.987885) (end 48.802762 -67.102484) (width 0.5) (layer "F.Cu") (net 2))
-  (segment (start 127.60785 -64.711491) (end 125.217087 -67.102254) (width 0.5) (layer "F.Cu") (net 2))
-  (segment (start 59.537571 -60.830584) (end 58.196209 -59.489222) (width 0.5) (layer "F.Cu") (net 2))
-  (segment (start 77.299673 -64.435238) (end 71.813295 -64.435238) (width 0.5) (layer "F.Cu") (net 2))
-  (segment (start 124.886497 -44.183183) (end 122.611414 -46.304732) (width 0.5) (layer "F.Cu") (net 2))
-  (segment (start 78.315672 -65.451237) (end 77.299673 -64.435238) (width 0.5) (layer "F.Cu") (net 2))
-  (segment (start 58.196209 -59.489222) (end 53.137791 -59.489222) (width 0.5) (layer "F.Cu") (net 2))
-  (segment (start 71.395635 -97.918702) (end 66.26837 -97.918702) (width 0.5) (layer "F.Cu") (net 2))
-  (segment (start 53.137791 -59.489222) (end 49.917361 -62.709652) (width 0.5) (layer "F.Cu") (net 2))
-  (segment (start 108.987449 -82.812254) (end 115.424791 -82.812254) (width 0.5) (layer "F.Cu") (net 2))
-  (segment (start 133.481554 -81.687254) (end 127.904087 -81.687254) (width 0.5) (layer "F.Cu") (net 2))
-  (segment (start 125.224525 -109.33275) (end 125.224525 -101.152875) (width 0.5) (layer "F.Cu") (net 2))
-  (segment (start 86.601289 -108.171928) (end 86.570217 -108.140856) (width 0.5) (layer "F.Cu") (net 2))
-  (segment (start 93.254215 -108.171928) (end 86.601289 -108.171928) (width 0.5) (layer "F.Cu") (net 2))
-  (segment (start 68.485407 -81.17697) (end 65.538664 -84.123713) (width 0.5) (layer "F.Cu") (net 2))
-  (segment (start 85.651298 -93.599163) (end 85.651298 -100.128683) (width 0.5) (layer "F.Cu") (net 2))
-  (segment (start 107.136087 -110.436017) (end 107.136087 -102.256142) (width 0.5) (layer "F.Cu") (net 2))
-  (segment (start 65.538664 -84.123713) (end 65.538664 -90.259425) (width 0.5) (layer "F.Cu") (net 2))
-  (segment (start 48.802762 -67.102484) (end 48.802762 -67.639549) (width 0.5) (layer "F.Cu") (net 2))
-  (segment (start 147.749135 -40.08246) (end 144.745631 -39.977575) (width 0.5) (layer "F.Cu") (net 2))
-  (segment (start 133.505791 -64.711491) (end 127.60785 -64.711491) (width 0.5) (layer "F.Cu") (net 2))
   (segment (start 154.256703 -114.199254) (end 150.44369 -114.199254) (width 0.5) (layer "F.Cu") (net 2))
-  (segment (start 115.424791 -65.812254) (end 109.709791 -65.812254) (width 0.5) (layer "F.Cu") (net 2))
-  (segment (start 122.611414 -46.304732) (end 122.314371 -54.810935) (width 0.5) (layer "F.Cu") (net 2))
-  (segment (start 125.217087 -84.374254) (end 125.217087 -92.335254) (width 0.5) (layer "F.Cu") (net 2))
-  (segment (start 127.668413 -98.708987) (end 133.513229 -98.708987) (width 0.5) (layer "F.Cu") (net 2))
-  (segment (start 94.735862 -91.236618) (end 88.013843 -91.236618) (width 0.5) (layer "F.Cu") (net 2))
-  (segment (start 48.232895 -75.218284) (end 44.864298 -78.586881) (width 0.5) (layer "F.Cu") (net 2))
-  (segment (start 87.132946 -76.929018) (end 87.132946 -83.193373) (width 0.5) (layer "F.Cu") (net 2))
-  (segment (start 129.462225 -44.342971) (end 124.886497 -44.183183) (width 0.5) (layer "F.Cu") (net 2))
-  (segment (start 88.013843 -91.236618) (end 85.651298 -93.599163) (width 0.5) (layer "F.Cu") (net 2))
   (segment (start 154.304587 -114.247138) (end 154.256703 -114.199254) (width 0.5) (layer "F.Cu") (net 2))
-  (segment (start 44.864298 -78.586881) (end 44.864298 -82.864875) (width 0.5) (layer "F.Cu") (net 2))
-  (segment (start 86.570217 -108.140856) (end 84.169651 -110.541422) (width 0.5) (layer "F.Cu") (net 2))
-  (segment (start 144.745631 -39.977575) (end 141.797987 -42.726297) (width 0.5) (layer "F.Cu") (net 2))
-  (segment (start 107.136087 -93.436017) (end 107.136087 -84.663616) (width 0.5) (layer "F.Cu") (net 2))
-  (segment (start 54.567252 -77.087765) (end 52.697771 -75.218284) (width 0.5) (layer "F.Cu") (net 2))
-  (segment (start 108.15356 -68.448217) (end 108.15356 -74.458485) (width 0.5) (layer "F.Cu") (net 2))
-  (segment (start 72.411634 -98.934701) (end 71.395635 -97.918702) (width 0.5) (layer "F.Cu") (net 2))
-  (segment (start 68.490683 -67.75785) (end 68.490683 -73.517693) (width 0.5) (layer "F.Cu") (net 2))
-  (segment (start 52.697771 -75.218284) (end 48.232895 -75.218284) (width 0.5) (layer "F.Cu") (net 2))
-  (segment (start 125.224525 -101.152875) (end 127.668413 -98.708987) (width 0.5) (layer "F.Cu") (net 2))
-  (segment (start 108.167264 -67.354781) (end 108.167264 -68.352254) (width 0.5) (layer "F.Cu") (net 2))
-  (segment (start 44.864298 -82.864875) (end 43.832443 -83.89673) (width 0.5) (layer "F.Cu") (net 2))
-  (segment (start 49.917361 -62.709652) (end 49.917361 -65.987885) (width 0.5) (layer "F.Cu") (net 2))
-  (segment (start 129.814449 -44.720686) (end 129.462225 -44.342971) (width 0.5) (layer "F.Cu") (net 2))
-  (segment (start 107.136087 -102.256142) (end 109.579975 -99.812254) (width 0.5) (layer "F.Cu") (net 2))
-  (segment (start 108.15356 -74.458485) (end 107.136087 -75.475958) (width 0.5) (layer "F.Cu") (net 2))
-  (segment (start 84.169651 -110.541422) (end 84.169651 -117.063993) (width 0.5) (layer "F.Cu") (net 2))
-  (segment (start 125.217087 -74.347787) (end 125.230791 -74.361491) (width 0.5) (layer "F.Cu") (net 2))
   (via (at 154.304587 -114.247138) (size 0.8) (drill 0.4) (layers "F.Cu" "B.Cu") (free) (net 2))
   (segment (start 154.329345 -114.22238) (end 154.352471 -114.199254) (width 0.5) (layer "B.Cu") (net 2))
@@
   (segment (start 159.239791 -76.162254) (end 158.159791 -76.162254) (width 0.5) (layer "B.Cu") (net 20))
   (segment (start 157.226791 -61.602254) (end 158.223791 -61.602254) (width 0.5) (layer "B.Cu") (net 20))
-  (zone (net 0) (net_name "") (layer "F.Cu") (hatch edge 0.508)
+  (zone (net 2) (net_name "GND") (layer "F.Cu") (hatch edge 0.508)
     (connect_pads (clearance 0.508))
     (min_thickness 0.254) (filled_areas_thickness no)
-    (fill yes (thermal_gap 0.508) (thermal_bridge_width 0.508))
+    (fill yes (thermal_gap 0.508) (thermal_bridge_width 0.508) (island_removal_mode 1) (island_area_min 0))
     (polygon
       (pts
