File: boards/wizza/wizza.kicad_pcb (KiCad board)
At the start: 2 copper layers, 106.6 x 85.9 mm, 27 parts

Commit message: wizza
Parts:
- moved REF** 1.93 mm to (104.2, -89.3), turned to 5 degrees
Routing:
- net P3: track 137.0 -> 135.6 mm
- net P14: track 103.3 -> 104.0 mm
