File: boards/basbousa/basbousa.kicad_pcb (KiCad board)
At the start: 2 copper layers, 133.4 x 90.7 mm, 25 parts

Commit message: clean up all the boards
Parts:
- moved S19 2.00 mm to (115.4, -70.7)
- moved S21 2.00 mm to (115.4, -87.7)
- moved S23 2.00 mm to (115.4, -104.7)
- moved S25 2.00 mm to (134.0, -69.2)
- moved S27 2.00 mm to (134.0, -86.2)
- moved S29 2.00 mm to (134.0, -103.2)
- moved REF** 0.51 mm to (103.6, -87.0)
Routing:
- net GND: track 315.1 -> 38.4 mm
- net P7: track 163.0 -> 161.0 mm
- net P6: track 146.7 -> 144.7 mm
- net P3: track 145.4 -> 144.3 mm
- net P0: track 142.4 -> 141.4 mm
- added copper zone on F.Cu, net GND

Commit message: basbousa new case with holes and chocV2 change
Parts:
- added ?: , , F.Cu at (40.4, -50.3)
- added ?: , , F.Cu at (131.1, -116.8)
- added ?: , , F.Cu at (60.5, -119.6)
- added ?: , , F.Cu at (148.8, -56.6)
Changed lines of the file:
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@@
       (net 2 "GND"))
   )
+  (footprint "" (layer "F.Cu")
+    (at 40.386 -50.292)
+    (fp_text reference "" (at 0 0) (layer "F.SilkS")
+      (effects (font (size 1.27 1.27) (thickness 0.15)))
+    )
+    (fp_text value "" (at 0 0) (layer "F.SilkS")
+      (effects (font (size 1.27 1.27) (thickness 0.15)))
+    )
+    (pad "1" thru_hole circle (at 0 0) (size 5 5) (drill 3) (layers *.Cu *.Mask)
+      (pinfunction "1") (pintype "input"))
+  )
   (footprint "Alaa:key" (layer "F.Cu")
     (at 133.985 -103.178)
@@
       (net 2 "GND"))
   )
+  (footprint "" (layer "F.Cu")
+    (at 131.064 -116.84)
+    (fp_text reference "" (at 0 0) (layer "F.SilkS")
+      (effects (font (size 1.27 1.27) (thickness 0.15)))
+    )
+    (fp_text value "" (at 0 0) (layer "F.SilkS")
+      (effects (font (size 1.27 1.27) (thickness 0.15)))
+    )
+    (pad "1" thru_hole circle (at 0 0) (size 5 5) (drill 3) (layers *.Cu *.Mask)
+      (pinfunction "1") (pintype "input"))
+  )
   (footprint "LOGO" (layer "F.Cu")
     (at 91.44 -50.8)
@@
       (net 2 "GND"))
   )
+  (footprint "" (layer "F.Cu")
+    (at 60.452 -119.634)
+    (fp_text reference "" (at 0 0) (layer "F.SilkS")
+      (effects (font (size 1.27 1.27) (thickness 0.15)))
+    )
+    (fp_text value "" (at 0 0) (layer "F.SilkS")
+      (effects (font (size 1.27 1.27) (thickness 0.15)))
+    )
+    (pad "1" thru_hole circle (at 0 0) (size 5 5) (drill 3) (layers *.Cu *.Mask)
+      (pinfunction "1") (pintype "input"))
+  )
   (footprint "Alaa:key" (layer "F.Cu")
     (at 96.386781 -80.178857 5)
@@
       (net 2 "GND"))
   )
+  (footprint "" (layer "F.Cu")
+    (at 148.844 -56.642)
+    (fp_text reference "" (at 0 0) (layer "F.SilkS")
+      (effects (font (size 1.27 1.27) (thickness 0.15)))
+    )
+    (fp_text value "" (at 0 0) (layer "F.SilkS")
+      (effects (font (size 1.27 1.27) (thickness 0.15)))
+    )
+    (pad "1" thru_hole circle (at 0 0) (size 5 5) (drill 3) (layers *.Cu *.Mask)
+      (pinfunction "1") (pintype "input"))
+  )
   (footprint "Alaa:key" (layer "F.Cu")
     (at 133.985 -69.178)
@@
   (gr_line (start 26.67 -58.928) (end 26.762446 -122.081554) (layer "Edge.Cuts") (width 0.15))
   (gr_arc (start 136.378 -124.477905) (mid 153.005122 -117.643705) (end 160.02 -101.092) (layer "Edge.Cuts") (width 0.15))
+  (gr_arc (start 26.762446 -122.081554) (mid 27.432001 -123.697999) (end 29.048446 -124.367554) (layer "Edge.Cuts") (width 0.15))
   (gr_arc (start 50.292 -33.794081) (mid 33.209738 -41.406869) (end 26.67 -58.928) (layer "Edge.Cuts") (width 0.15))
   (gr_arc (start 160.00102 -36.322) (mid 159.230194 -34.525146) (end 157.426728 -33.769919) (layer "Edge.Cuts") (width 0.15))
   (gr_line (start 160.00102 -36.322) (end 160.02 -101.092) (layer "Edge.Cuts") (width 0.15))
   (gr_line (start 157.426728 -33.769919) (end 50.292 -33.794081) (layer "Edge.Cuts") (width 0.15))
-  (gr_arc (start 26.762446 -122.081554) (mid 27.432 -123.698) (end 29.048446 -124.367554) (layer "Edge.Cuts") (width 0.15))
   (segment (start 118.536566 -76.486496) (end 118.536566 -68.760538) (width 0.25) (layer "F.Cu") (net 1))
   (segment (start 67.64256 -67.868594) (end 73.906114 -61.60504) (width 0.25) (layer "F.Cu") (net 1))
