File: boards/30keys/battoota/battoota.kicad_pcb (KiCad board)
At the start: 2 copper layers, 122.6 x 88.9 mm, 23 parts

Commit message: new cases for konafa and battoota
Parts:
- added ?: , , F.Cu at (50.1, -115.2)
- added ?: , , F.Cu at (49.1, -40.8)
- added ?: , , F.Cu at (159.1, -38.5)
- moved S31 1.00 mm to (132.0, -51.5)
- moved S33 1.00 mm to (151.2, -45.8)
Routing:
- net P9: track 76.4 -> 73.6 mm
- net P8: track 84.1 -> 85.4 mm
Changed lines of the file:
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@@
       (net 2 "GND"))
+  )
+  (footprint "" (layer "F.Cu")
+    (at 50.146791 -115.215254)
+    (fp_text reference "" (at 0 0) (layer "F.SilkS")
+      (effects (font (size 1.27 1.27) (thickness 0.15)))
+    )
+    (fp_text value "" (at 0 0) (layer "F.SilkS")
+      (effects (font (size 1.27 1.27) (thickness 0.15)))
+    )
+    (pad "1" thru_hole circle (at 0 0) (size 5 5) (drill 3) (layers *.Cu *.Mask)
+      (pinfunction "1") (pintype "input"))
   )
   (footprint "LOGO" (layer "F.Cu")
@@
   )
   (footprint "Alaa:choc_hotswap_key" (layer "F.Cu")
-    (at 152.214001 -45.787044 -24)
+    (at 151.214001 -45.787044 -24)
     (attr through_hole)
     (fp_text reference "S33" (at 0 0 139) (layer "F.SilkS") hide
@@
       (net 2 "GND"))
   )
+  (footprint "" (layer "F.Cu")
+    (at 49.130791 -40.793254)
+    (fp_text reference "" (at 0 0) (layer "F.SilkS")
+      (effects (font (size 1.27 1.27) (thickness 0.15)))
+    )
+    (fp_text value "" (at 0 0) (layer "F.SilkS")
+      (effects (font (size 1.27 1.27) (thickness 0.15)))
+    )
+    (pad "1" thru_hole circle (at 0 0) (size 5 5) (drill 3) (layers *.Cu *.Mask)
+      (pinfunction "1") (pintype "input"))
+  )
   (footprint "Alaa:choc_hotswap_key" (layer "F.Cu")
-    (at 132.975328 -51.485799 -9)
+    (at 131.975328 -51.485799 -9)
     (attr through_hole)
     (fp_text reference "S31" (at 0 0 154) (layer "F.SilkS") hide
@@
     (pad "2" smd rect (at 8.275 -3.749999 17) (size 2.6 2.6) (layers "B.Cu" "B.Paste" "B.Mask")
       (net 2 "GND"))
+  )
+  (footprint "" (layer "F.Cu")
+    (at 159.112791 -38.507254)
+    (fp_text reference "" (at 0 0) (layer "F.SilkS")
+      (effects (font (size 1.27 1.27) (thickness 0.15)))
+    )
+    (fp_text value "" (at 0 0) (layer "F.SilkS")
+      (effects (font (size 1.27 1.27) (thickness 0.15)))
+    )
+    (pad "1" thru_hole circle (at 0 0) (size 5 5) (drill 3) (layers *.Cu *.Mask)
+      (pinfunction "1") (pintype "input"))
   )
   (footprint "Alaa:Tenting_Puck_3_Holes" (layer "F.Cu")
@@
   (segment (start 155.527414 -71.97371) (end 155.191874 -71.638171) (width 0.25) (layer "F.Cu") (net 16))
   (segment (start 161.977213 -91.442348) (end 157.969791 -91.442348) (width 0.25) (layer "F.Cu") (net 16))
+  (segment (start 136.339001 -56.048429) (end 134.942686 -54.652114) (width 0.25) (layer "F.Cu") (net 16))
   (segment (start 147.665453 -64.111751) (end 137.981288 -64.111751) (width 0.25) (layer "F.Cu") (net 16))
-  (segment (start 137.319319 -47.981726) (end 137.319319 -46.950411) (width 0.25) (layer "F.Cu") (net 16))
-  (segment (start 136.339001 -48.962044) (end 137.319319 -47.981726) (width 0.25) (layer "F.Cu") (net 16))
-  (segment (start 127.630147 -48.327044) (end 127.442436 -48.514755) (width 0.25) (layer "F.Cu") (net 16))
   (segment (start 137.140791 -63.271254) (end 137.140791 -56.850221) (width 0.25) (layer "F.Cu") (net 16))
+  (segment (start 134.942686 -48.327044) (end 126.630147 -48.327044) (width 0.25) (layer "F.Cu") (net 16))
   (segment (start 155.527414 -71.973711) (end 155.191874 -71.638171) (width 0.25) (layer "F.Cu") (net 16))
+  (segment (start 134.942686 -49.977359) (end 136.319319 -48.600726) (width 0.25) (layer "F.Cu") (net 16))
+  (segment (start 136.319319 -46.950411) (end 134.942686 -48.327044) (width 0.25) (layer "F.Cu") (net 16))
   (segment (start 155.527414 -88.999971) (end 155.527414 -71.973711) (width 0.25) (layer "F.Cu") (net 16))
-  (segment (start 137.319319 -46.950411) (end 135.942686 -48.327044) (width 0.25) (layer "F.Cu") (net 16))
-  (segment (start 135.942686 -48.327044) (end 127.630147 -48.327044) (width 0.25) (layer "F.Cu") (net 16))
+  (segment (start 136.319319 -48.600726) (end 136.319319 -46.950411) (width 0.25) (layer "F.Cu") (net 16))
+  (segment (start 134.942686 -54.652114) (end 134.942686 -49.977359) (width 0.25) (layer "F.Cu") (net 16))
   (segment (start 137.981288 -64.111751) (end 137.140791 -63.271254) (width 0.25) (layer "F.Cu") (net 16))
-  (segment (start 136.339001 -56.048429) (end 136.339001 -48.962044) (width 0.25) (layer "F.Cu") (net 16))
   (segment (start 155.191874 -71.638171) (end 147.665453 -64.111751) (width 0.25) (layer "F.Cu") (net 16))
   (segment (start 157.969791 -91.442348) (end 155.527414 -88.999971) (width 0.25) (layer "F.Cu") (net 16))
-  (segment (start 127.442435 -49.590478) (end 127.442435 -48.514756) (width 0.25) (layer "B.Cu") (net 16))
-  (segment (start 130.671434 -57.874867) (end 130.671434 -52.819477) (width 0.25) (layer "B.Cu") (net 16))
-  (segment (start 130.671434 -52.819477) (end 127.442435 -49.590478) (width 0.25) (layer "B.Cu") (net 16))
-  (segment (start 155.976934 -55.359111) (end 157.625944 -53.710101) (width 0.25) (layer "F.Cu") (net 17))
-  (segment (start 155.389001 -40.43476) (end 155.236129 -40.281888) (width 0.25) (layer "F.Cu") (net 17))
+  (segment (start 130.671434 -54.007897) (end 126.442435 -49.778898) (width 0.25) (layer "B.Cu") (net 16))
+  (segment (start 126.442435 -49.778898) (end 126.442435 -48.514756) (width 0.25) (layer "B.Cu") (net 16))
+  (segment (start 130.671434 -56.874867) (end 130.671434 -54.007897) (width 0.25) (layer "B.Cu") (net 16))
+  (segment (start 129.671433 -57.874868) (end 130.671434 -56.874867) (width 0.25) (layer "B.Cu") (net 16))
+  (segment (start 155.976934 -86.909491) (end 155.976934 -50.539586) (width 0.25) (layer "F.Cu") (net 17))
+  (segment (start 155.976934 -50.539586) (end 156.625944 -49.890576) (width 0.25) (layer "F.Cu") (net 17))
+  (segment (start 154.236129 -47.500761) (end 154.236129 -41.281888) (width 0.25) (layer "F.Cu") (net 17))
+  (segment (start 153.274157 -40.281888) (end 149.206791 -44.349254) (width 0.25) (layer "F.Cu") (net 17))
+  (segment (start 149.206791 -44.349254) (end 146.100675 -44.349254) (width 0.25) (layer "F.Cu") (net 17))
   (segment (start 161.977213 -88.902348) (end 157.969791 -88.902348) (width 0.25) (layer "F.Cu") (net 17))
+  (segment (start 156.625945 -49.890577) (end 154.236129 -47.500761) (width 0.25) (layer "F.Cu") (net 17))
   (segment (start 157.969791 -88.902348) (end 155.976934 -86.909491) (width 0.25) (layer "F.Cu") (net 17))
-  (segment (start 155.389001 -47.653633) (end 155.389001 -40.43476) (width 0.25) (layer "F.Cu") (net 17))
-  (segment (start 157.625944 -53.710101) (end 157.625944 -49.890576) (width 0.25) (layer "F.Cu") (net 17))
-  (segment (start 153.274157 -40.281888) (end 149.206791 -44.349254) (width 0.25) (layer "F.Cu") (net 17))
-  (segment (start 155.236129 -40.281888) (end 153.274157 -40.281888) (width 0.25) (layer "F.Cu") (net 17))
-  (segment (start 149.206791 -44.349254) (end 146.100675 -44.349254) (width 0.25) (layer "F.Cu") (net 17))
-  (segment (start 155.976934 -86.909491) (end 155.976934 -55.359111) (width 0.25) (layer "F.Cu") (net 17))
-  (segment (start 157.625945 -49.890577) (end 155.389001 -47.653633) (width 0.25) (layer "F.Cu") (net 17))
-  (segment (start 151.642223 -52.554701) (end 151.642223 -50.295266) (width 0.25) (layer "B.Cu") (net 17))
-  (segment (start 151.642223 -50.295266) (end 146.100675 -44.753718) (width 0.25) (layer "B.Cu") (net 17))
+  (segment (start 154.236129 -40.281888) (end 153.274157 -40.281888) (width 0.25) (layer "F.Cu") (net 17))
+  (segment (start 150.642222 -49.295265) (end 146.100675 -44.753718) (width 0.25) (layer "B.Cu") (net 17))
+  (segment (start 150.642222 -52.554702) (end 150.642222 -49.295265) (width 0.25) (layer "B.Cu") (net 17))
   (segment (start 146.100675 -44.753718) (end 146.100675 -44.349254) (width 0.25) (layer "B.Cu") (net 17))
   (segment (start 152.372041 -116.88499) (end 150.419502 -116.88499) (width 0.5) (layer "F.Cu") (net 18))

Commit message: change areas for better pictures
Changed lines of the file:
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@@
   (segment (start 135.118406 -112.746869) (end 135.109791 -112.738254) (width 0.5) (layer "B.Cu") (net 20))
   (segment (start 135.118406 -118.676838) (end 135.118406 -112.746869) (width 0.5) (layer "B.Cu") (net 20))
-  (zone (net 2) (net_name "GND") (layer "F.Cu") (hatch edge 0.508)
+  (zone (net 2) (net_name "GND") (layers F&B.Cu) (hatch edge 0.508)
     (connect_pads (clearance 0.508))
     (min_thickness 0.254) (filled_areas_thickness no)
@@
     (polygon
       (pts
-        (xy 176.511791 -127.788254)
-        (xy 176.765791 -127.788254)
-        (xy 175.495791 -28.601254)
-        (xy 22.333791 -27.331254)
-        (xy 24.619791 -130.201254)
+        (xy 164.954791 -124.105254)
+        (xy 164.700791 -124.105254)
+        (xy 164.954791 -32.157254)
+        (xy 39.986791 -32.411254)
+        (xy 40.240791 -124.613254)
       )
     )
-  )
-  (zone locked (net 2) (net_name "GND") (layer "B.Cu") (hatch edge 0.508)
-    (connect_pads (clearance 0.508))
-    (min_thickness 0.254) (filled_areas_thickness no)
-    (fill yes (thermal_gap 0.508) (thermal_bridge_width 0.508))
-    (polygon
-      (pts
-        (xy 185.274791 -132.868254)
-        (xy 188.341 -13.2842)
-        (xy 15.094791 -16.028254)
-        (xy 12.554791 -132.868254)
-        (xy 86.7918 -132.868254)
-      )
-    )
