File: boards/30keys/battoota_min/battoota_min.kicad_pcb (KiCad board)
At the start: 2 copper layers, 108.4 x 82.1 mm, 21 parts

Commit message: change areas for better pictures
Changed lines of the file:
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@@
     (polygon
       (pts
-        (xy 322.199 50.038)
-        (xy 313.309 152.273)
-        (xy 175.387 153.289)
-        (xy 179.197 49.784)
+        (xy 302.641 55.753)
+        (xy 300.863 141.859)
+        (xy 188.087 140.589)
+        (xy 188.849 55.499)
       )
     )
