File: boards/30keys/wizza/wizza.kicad_pcb (KiCad board)
At the start: 2 copper layers, 106.6 x 85.9 mm, 27 parts

Commit message: change areas for better pictures
Changed lines of the file:
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@@
     (polygon
       (pts
-        (xy 185.274791 -132.868254)
-        (xy 188.341 -13.2842)
-        (xy 15.094791 -16.028254)
-        (xy 12.554791 -132.868254)
-        (xy 86.7918 -132.868254)
+        (xy 152.000791 -31.903254)
+        (xy 38.716791 -31.903254)
+        (xy 38.716791 -125.883254)
+        (xy 152.254791 -125.883254)
       )
     )
