File: boards/32keys/konafa/konafa.kicad_pcb (KiCad board)
At the start: 2 copper layers, 122.6 x 88.9 mm, 28 parts

Commit message: change areas for better pictures
Changed lines of the file:
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@@
   (segment (start 159.239791 -76.162254) (end 158.159791 -76.162254) (width 0.5) (layer "B.Cu") (net 20))
   (segment (start 157.226791 -61.602254) (end 158.223791 -61.602254) (width 0.5) (layer "B.Cu") (net 20))
-  (zone (net 2) (net_name "GND") (layer "F.Cu") (hatch edge 0.508)
+  (zone (net 2) (net_name "GND") (layers F&B.Cu) (hatch edge 0.508)
     (connect_pads (clearance 0.508))
     (min_thickness 0.254) (filled_areas_thickness no)
@@
     (polygon
       (pts
-        (xy 186.036791 -15.901254)
-        (xy 18.142791 -18.187254)
-        (xy 14.713791 -130.582254)
-        (xy 184.004791 -131.217254)
+        (xy 165.208791 -32.919254)
+        (xy 39.986791 -31.903254)
+        (xy 39.224791 -124.613254)
+        (xy 166.478791 -124.359254)
       )
     )
-  )
-  (zone (net 2) (net_name "GND") (layer "B.Cu") (hatch edge 0.508)
-    (connect_pads (clearance 0.508))
-    (min_thickness 0.254) (filled_areas_thickness no)
-    (fill yes (thermal_gap 0.508) (thermal_bridge_width 0.508))
-    (polygon
-      (pts
-        (xy 185.274791 -132.868254)
-        (xy 188.341 -13.2842)
-        (xy 15.094791 -16.028254)
-        (xy 12.554791 -132.868254)
-        (xy 86.7918 -132.868254)
-      )
-    )
