File: boards/32keys/konafa_min/konafa_min.kicad_pcb (KiCad board)
At the start: 2 copper layers, 110.9 x 82.1 mm, 22 parts

Commit message: change areas for better pictures
Changed lines of the file:
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@@
     (polygon
       (pts
-        (xy 322.199 50.038)
-        (xy 313.309 152.273)
-        (xy 175.387 153.289)
-        (xy 179.197 49.784)
+        (xy 305.689 54.991)
+        (xy 304.165 142.621)
+        (xy 188.087 141.351)
+        (xy 189.103 54.483)
       )
     )
