File: boards/34keys/basbousa/basbousa.kicad_pcb (KiCad board)
At the start: 2 copper layers, 133.4 x 90.7 mm, 29 parts

Commit message: change areas for better pictures
Changed lines of the file:
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@@
     (polygon
       (pts
-        (xy 184.658 -135.128)
-        (xy 188.341 -13.2842)
-        (xy 1.524 -15.494)
-        (xy 0 -134.62)
-        (xy 88.265 -135.89)
+        (xy 161.29 -126.238)
+        (xy 163.576 -30.988)
+        (xy 24.384 -32.258)
+        (xy 24.13 -127.762)
+        (xy 90.678 -127.762)
       )
     )
