File: boards/36keys/basbousa36/basbousa.kicad_pcb (KiCad board)
At the start: 2 copper layers, 133.4 x 90.7 mm, 30 parts

Commit message: change areas for better pictures
Changed lines of the file:
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@@
       (effects (font (size 1.27 1.27) (thickness 0.15)))
     )
-    (fp_line (start -6.999999 7.000001) (end -7 6) (layer "Dwgs.User") (width 0.15))
     (fp_line (start -7 -5.999999) (end -7 -6.999999) (layer "Dwgs.User") (width 0.15))
+    (fp_line (start -6.999999 7.000001) (end -7 6) (layer "Dwgs.User") (width 0.15))
+    (fp_line (start -7 -6) (end -7 -7) (layer "Dwgs.User") (width 0.15))
     (fp_line (start 7 -7) (end 7 -6) (layer "Dwgs.User") (width 0.15))
+    (fp_line (start 6.999999 -7) (end 6 -6.999999) (layer "Dwgs.User") (width 0.15))
     (fp_line (start -9 -8.499999) (end 8.999999 -8.5) (layer "Dwgs.User") (width 0.15))
     (fp_line (start 6.999999 -7) (end 7 -5.999999) (layer "Dwgs.User") (width 0.15))
@@
     (fp_line (start 6 7) (end 7 7) (layer "Dwgs.User") (width 0.15))
     (fp_line (start 7 6) (end 7 7) (layer "Dwgs.User") (width 0.15))
-    (fp_line (start -9 8.5) (end -9 -8.5) (layer "Dwgs.User") (width 0.15))
     (fp_line (start 9 8.5) (end -8.999999 8.500001) (layer "Dwgs.User") (width 0.15))
+    (fp_line (start 9 8.5) (end -9 8.5) (layer "Dwgs.User") (width 0.15))
     (fp_line (start 9 -8.5) (end 9 8.5) (layer "Dwgs.User") (width 0.15))
     (fp_line (start -6 -7) (end -7 -7) (layer "Dwgs.User") (width 0.15))
     (fp_line (start -6 -6.999998) (end -7 -6.999999) (layer "Dwgs.User") (width 0.15))
-    (fp_line (start 6.999999 -7) (end 6 -6.999999) (layer "Dwgs.User") (width 0.15))
     (fp_line (start -8.999999 8.500001) (end -9 -8.499999) (layer "Dwgs.User") (width 0.15))
-    (fp_line (start -7 -6) (end -7 -7) (layer "Dwgs.User") (width 0.15))
     (fp_line (start 7 -7) (end 6 -7) (layer "Dwgs.User") (width 0.15))
+    (fp_line (start 6 7) (end 7 7) (layer "Dwgs.User") (width 0.15))
     (fp_line (start 7 6.000001) (end 7 7) (layer "Dwgs.User") (width 0.15))
+    (fp_line (start -9 8.5) (end -9 -8.5) (layer "Dwgs.User") (width 0.15))
     (fp_line (start -7 7) (end -7 6) (layer "Dwgs.User") (width 0.15))
-    (fp_line (start 6 7) (end 7 7) (layer "Dwgs.User") (width 0.15))
-    (fp_line (start 9 8.5) (end -9 8.5) (layer "Dwgs.User") (width 0.15))
     (pad "" np_thru_hole circle (at 5 -3.749999 343) (size 3 3) (drill 3) (layers *.Cu *.Mask)
       (net 10 "P15"))
@@
     (polygon
       (pts
-        (xy 184.658 -135.128)
-        (xy 188.341 -13.2842)
-        (xy 1.524 -15.494)
-        (xy 0 -134.62)
-        (xy 88.265 -135.89)
+        (xy 162.052 -126.492)
+        (xy 163.322 -31.75)
+        (xy 22.352 -30.734)
+        (xy 22.86 -128.524)
+        (xy 87.63 -128.016)
       )
     )
