File: boards/32keys/battoota-3thumb/battoota.kicad_pcb (KiCad board)
At the start: 2 copper layers, 122.6 x 88.9 mm, 24 parts

Commit message: battota preview
Changed lines of the file:
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@@
   (segment (start 137.133791 -54.282161) (end 137.133791 -47.029997) (width 0.25) (layer "F.Cu") (net 16))
   (segment (start 131.454491 -56.985868) (end 132.343492 -56.096867) (width 0.25) (layer "B.Cu") (net 16))
-  (segment (start 129.114494 -49.537957) (end 129.114494 -47.625755) (width 0.25) (layer "B.Cu") (net 16))
   (segment (start 132.343492 -56.096867) (end 132.343492 -52.766955) (width 0.25) (layer "B.Cu") (net 16))
   (segment (start 132.343492 -52.766955) (end 129.114494 -49.537957) (width 0.25) (layer "B.Cu") (net 16))
+  (segment (start 129.114494 -49.537957) (end 129.114494 -47.625755) (width 0.25) (layer "B.Cu") (net 16))
   (segment (start 161.977213 -88.902348) (end 157.969791 -88.902348) (width 0.25) (layer "F.Cu") (net 17))
   (segment (start 158.409003 -49.001577) (end 156.437791 -47.030365) (width 0.25) (layer "F.Cu") (net 17))
@@
   (segment (start 135.118406 -112.746869) (end 135.109791 -112.738254) (width 0.5) (layer "B.Cu") (net 20))
   (segment (start 135.118406 -118.676838) (end 135.118406 -112.746869) (width 0.5) (layer "B.Cu") (net 20))
-  (zone (net 2) (net_name "GND") (layer "F.Cu") (hatch edge 0.508)
+  (zone (net 2) (net_name "GND") (layers F&B.Cu) (hatch edge 0.508)
     (connect_pads (clearance 0.508))
     (min_thickness 0.254) (filled_areas_thickness no)
@@
     (polygon
       (pts
-        (xy 176.511791 -127.788254)
-        (xy 176.765791 -127.788254)
-        (xy 175.495791 -28.601254)
-        (xy 22.333791 -27.331254)
-        (xy 24.619791 -130.201254)
+        (xy 166.732791 -125.121254)
+        (xy 166.732791 -125.121254)
+        (xy 165.208791 -31.903254)
+        (xy 38.462791 -31.903254)
+        (xy 38.462791 -125.883254)
       )
     )
-  )
-  (zone locked (net 2) (net_name "GND") (layer "B.Cu") (hatch edge 0.508)
-    (connect_pads (clearance 0.508))
-    (min_thickness 0.254) (filled_areas_thickness no)
-    (fill yes (thermal_gap 0.508) (thermal_bridge_width 0.508))
-    (polygon
-      (pts
-        (xy 185.274791 -132.868254)
-        (xy 188.341 -13.2842)
-        (xy 15.094791 -16.028254)
-        (xy 12.554791 -132.868254)
-        (xy 86.7918 -132.868254)
-      )
-    )
