File: boards/30keys/Asfoora/Asfoora.kicad_sch (KiCad schematic)
At the start: 70 parts, among them J1 Conn_01x12_Female, SW1 Rotary_Encoder_Switch, SW10 SW_Push, SW11 SW_Push, SW12 SW_Push, SW13 SW_Push, SW14 SW_Push, SW15 SW_Push, SW16 Rotary_Encoder_Switch, SW17 SW_Push, SW18 SW_Push, SW19 SW_Push, SW2 SW_Push, SW20 SW_Push, SW21 SW_Push, SW22 SW_Push, SW23 SW_Push, SW24 SW_Push, SW25 SW_Push, SW26 SW_Push, SW27 SW_Push, SW28 SW_Push, SW29 SW_Push, SW3 SW_Push, SW30 SW_Push, SW31 SW_Push, SW32 SW_Push, SW33 SW_Push, SW34 SW_SPDT, SW4 SW_Push, SW5 SW_Push, SW6 SW_Push, SW7 SW_Push, SW8 SW_Push, SW9 SW_Push

Commit message: Asfoora
Parts:
- D1, D10, D11, D12, D13, D14, D15, D16, D17, D18, D19, D2, D20, D21, D22, D23, D24, D25, D26, D27, D28, D29, D3, D30, D31, D32, D4, D5, D6, D7, D8, D9: symbol Diode:1N4148 -> alaa:Diode_1N4148; LCSC (none) -> C909967
- J1: LCSC (none) -> C479750
- R1, R2: symbol Device:R -> alaa:4k7; LCSC (none) -> C269746
- U1: value (none) -> ProMicro_r; footprint (none) -> kbd:ProMicro_v3.5

Commit message: asfoora changes
Connections:
- net SW31A renamed row_2
- net SW31B: no longer names the net of D15.2 (A), SW1.S2
- net SW32B: no longer names the net of D19.2 (A), SW16.S1
Other:
- moved on the sheet: SW1, SW16
