File: boards/30keys/wizza-mx/wizza.kicad_pcb (KiCad board)
At the start: 2 copper layers, 110.2 x 90.6 mm, 27 parts

Commit message: update asfoora and wizza mx
Parts:
- S1, S10, S11, S12, S13, S14, S15, S2, S3, S4, S5, S6, S7, S8, S9: footprint Alaa:MX -> Alaa:MX-hotswap-reversible
Routing:
- net matrix_pinky_top: track 60.2 -> 52.0 mm
- net matrix_pinky_home: track 41.0 -> 32.8 mm
- net matrix_ring_home: track 67.1 -> 59.1 mm
- net matrix_ring_top: track 84.7 -> 76.6 mm
- net matrix_ring_bottom: track 47.7 -> 39.6 mm
- net matrix_middle_home: track 88.7 -> 80.9 mm
- net matrix_middle_bottom: track 71.3 -> 63.4 mm
- net matrix_inner_home: track 144.7 -> 137.1 mm
- net matrix_inner_bottom: track 122.5 -> 114.9 mm
- net thumb_reachy: track 95.6 -> 87.9 mm
- net thumb_tucky: track 78.5 -> 70.8 mm
- net matrix_index_top: track 142.2 -> 134.6 mm
- net matrix_index_home: track 124.1 -> 116.4 mm
- net matrix_index_bottom: track 103.4 -> 95.8 mm
- net matrix_middle_top: track 111.9 -> 105.0 mm
