File: boards/30keys/wizza-mx/wizza.kicad_pcb (KiCad board)
At the start: 2 copper layers, 110.2 x 90.6 mm, 27 parts

Commit message: Wizza with better on off switch
Parts:
- removed T1, T2: , E73:SPDT_C128955
- added SW37: SW_SPDT, Alaa:SW_CuK_OS102011MA1QN1_SPDT_Angled, F.Cu at (206.6, 58.9)
Routing:
- net b+: track 45.0 -> 25.4 mm
- net RAW: track 94.9 -> 94.5 mm, vias 2 -> 1

Commit message: Gerber for wizza MX
Routing:
- net b+: track 25.4 -> 24.3 mm
- net GND: vias 1 -> 2
Changed lines of the file:
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@@
     (stroke (width 0.15) (type solid)) (layer "Edge.Cuts"))
   (segment (start 201.422 137.954) (end 201.422 141.867523) (width 0.5) (layer "F.Cu") (net 1))
+  (via (at 203.3 68.8) (size 0.8) (drill 0.4) (layers "F.Cu" "B.Cu") (free) (net 1))
   (via (at 201.422 137.922) (size 0.8) (drill 0.4) (layers "F.Cu" "B.Cu") (free) (net 1))
   (segment (start 201.422 134.117523) (end 201.422 137.954) (width 0.5) (layer "B.Cu") (net 1))
@@
   (segment (start 200.406 71.31) (end 200.406 67.564) (width 0.5) (layer "F.Cu") (net 19))
   (segment (start 204.68 67.12) (end 206.55 65.25) (width 0.5) (layer "F.Cu") (net 19))
-  (segment (start 206.55 65.25) (end 206.55 64.1) (width 0.5) (layer "F.Cu") (net 19))
   (zone (net 1) (net_name "GND") (layers "F&B.Cu") (hatch edge 0.508)
     (connect_pads (clearance 0.508))
     (min_thickness 0.254) (filled_areas_thickness no)
-    (fill yes (thermal_gap 0.508) (thermal_bridge_width 0.508) (island_removal_mode 1) (island_area_min 0))
+    (fill yes (thermal_gap 0.508) (thermal_bridge_width 0.508))
     (polygon
       (pts
