File: boards/30keys/wizza-chocV2/wizza.kicad_pcb (KiCad board)
At the start: 2 copper layers, 110.2 x 90.6 mm, 25 parts

Commit message: add logo to choc V2 board
Parts:
- added G***: LOGO, LOGO, F.Cu at (247.5, 131.0)
- added G***: LOGO, LOGO, B.Cu at (247.5, 131.0)
