File: boards/30keys/Batreeq/Batreeq.kicad_sch (KiCad schematic)
At the start: 96 parts, among them J1 Conn_01x12_Female, J2 Conn_01x12_Female, SW1 SW_Push, SW10 SW_Push, SW11 SW_Push, SW12 SW_Push, SW13 SW_Push, SW14 SW_Push, SW15 SW_Push, SW16 SW_Push, SW17 SW_Push, SW18 SW_Push, SW19 SW_Push, SW2 SW_Push, SW20 SW_Push, SW21 SW_Push, SW22 SW_Push, SW23 SW_Push, SW24 SW_Push, SW25 SW_Push, SW26 SW_Push, SW27 SW_Push, SW28 SW_Push, SW29 SW_Push, SW3 SW_Push, SW30 SW_Push, SW31 SW_Push, SW32 SW_Push, SW33 SW_Push, SW34 SW_Push, SW35 SW_Push, SW36 RotaryEncoder, SW37 SW_SPDT, SW4 SW_Push, SW5 SW_Push, SW6 SW_Push, SW7 SW_Push, SW8 SW_Push, SW9 SW_Push, U1 ProMicro_r, U2 74HC595, U3 TCR2EF19,LM(CT, U4 PMW3360DM-T2QU, U5 DRV2605L

Commit message: correct diode direction
Connections:
- net col0: now also D1.2 (A), D2.2 (A), D3.2 (A); no longer D1.1 (K), D2.1 (K), D3.1 (K)
- net col1: now also D4.2 (A), D5.2 (A), D6.2 (A), D7.2 (A); no longer D4.1 (K), D5.1 (K), D6.1 (K), D7.1 (K)
- net col2: now also D10.2 (A), D11.2 (A), D12.2 (A), D8.2 (A), D9.2 (A); no longer D10.1 (K), D11.1 (K), D12.1 (K), D8.1 (K), D9.1 (K)
- net col3: now also D13.2 (A), D14.2 (A), D15.2 (A), D16.2 (A), D17.2 (A); no longer D13.1 (K), D14.1 (K), D15.1 (K), D16.1 (K), D17.1 (K)
- net col4: now also D18.2 (A), D19.2 (A), D20.2 (A), D21.2 (A), D22.2 (A); no longer D18.1 (K), D19.1 (K), D20.1 (K), D21.1 (K), D22.1 (K)
- net col5: now also D23.2 (A), D24.2 (A), D25.2 (A), D26.2 (A), D27.2 (A); no longer D23.1 (K), D24.1 (K), D25.1 (K), D26.1 (K), D27.1 (K)
- net col6: now also D28.2 (A), D29.2 (A), D30.2 (A), D31.2 (A); no longer D28.1 (K), D29.1 (K), D30.1 (K), D31.1 (K)
- net col7: now also D32.2 (A), D33.2 (A), D34.2 (A); no longer D32.1 (K), D33.1 (K), D34.1 (K)
- net at SW4.2: now also D4.1 (K); no longer D4.2 (A)
- net at SW3.2: now also D3.1 (K); no longer D3.2 (A)
- net at SW19.2: now also D19.1 (K); no longer D19.2 (A)
- net at SW29.2: now also D29.1 (K); no longer D29.2 (A)
- net at SW1.2: now also D1.1 (K); no longer D1.2 (A)
- net at SW31.2: now also D31.1 (K); no longer D31.2 (A)
- net at SW12.2: now also D12.1 (K); no longer D12.2 (A)
- net at SW26.2: now also D26.1 (K); no longer D26.2 (A)
- net at SW28.2: now also D28.1 (K); no longer D28.2 (A)
- net at SW5.2: now also D5.1 (K); no longer D5.2 (A)
- net at SW17.2: now also D17.1 (K); no longer D17.2 (A)
- net at SW15.2: now also D15.1 (K); no longer D15.2 (A)
- net at SW24.2: now also D24.1 (K); no longer D24.2 (A)
- net at SW21.2: now also D21.1 (K); no longer D21.2 (A)
- net at SW11.2: now also D11.1 (K); no longer D11.2 (A)
- net at SW27.2: now also D27.1 (K); no longer D27.2 (A)
- net at SW8.2: now also D8.1 (K); no longer D8.2 (A)
- net at SW23.2: now also D23.1 (K); no longer D23.2 (A)
- net at SW6.2: now also D6.1 (K); no longer D6.2 (A)
- net at SW32.2: now also D32.1 (K); no longer D32.2 (A)
- net at SW18.2: now also D18.1 (K); no longer D18.2 (A)
- net at SW20.2: now also D20.1 (K); no longer D20.2 (A)
- net at SW22.2: now also D22.1 (K); no longer D22.2 (A)
- net at SW10.2: now also D10.1 (K); no longer D10.2 (A)
- net at SW13.2: now also D13.1 (K); no longer D13.2 (A)
- net at SW14.2: now also D14.1 (K); no longer D14.2 (A)
- net at SW34.2: now also D34.1 (K); no longer D34.2 (A)
- net at SW9.2: now also D9.1 (K); no longer D9.2 (A)
- net at SW33.2: now also D33.1 (K); no longer D33.2 (A)
- net at SW30.2: now also D30.1 (K); no longer D30.2 (A)
- net at SW16.2: now also D16.1 (K); no longer D16.2 (A)
- net at SW7.2: now also D7.1 (K); no longer D7.2 (A)
- net at SW2.2: now also D2.1 (K); no longer D2.2 (A)
- net at SW25.2: now also D25.1 (K); no longer D25.2 (A)
Other:
- moved on the sheet: D10, D11, D12, D13, D14, D15, D16, D17, D18, D19, D2, D20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

Commit message: fix batreeq bodge and mcu footprint
Parts:
- U1: value ProMicro_r -> (none); footprint kbd:ProMicro_v3.5 -> (none)
Connections:
- net SCLK: now also U2.11 (SRCLK)
- net SRCLK: no longer names the net of U1.17 (A0/F7)
- net SRCLK: no longer U2.11 (SRCLK)
- no-connect marks 14 -> 15
Changed lines of the file:
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@@
   (no_connect (at 366.014 170.942))
   (no_connect (at 272.288 114.3))
+  (no_connect (at 249.682 62.23))
   (no_connect (at 249.682 59.69))
   (no_connect (at 272.288 104.14))
@@
     )
   )
-  (global_label "SRCLK" (shape input) (at 249.682 62.23 0) (fields_autoplaced)
-    (effects (font (size 1.27 1.27)) (justify left))
-    (property "Intersheet References" "${INTERSHEET_REFS}" (id 0) (at 258.1427 62.1506 0)
-      (effects (font (size 1.27 1.27)) (justify left) hide)
-    )
-  )
   (global_label "MOTION" (shape input) (at 272.288 119.38 180) (fields_autoplaced)
     (effects (font (size 1.27 1.27)) (justify right))
@@
     )
   )
-  (global_label "SRCLK" (shape input) (at 218.694 106.426 180) (fields_autoplaced)
+  (global_label "SCLK" (shape input) (at 218.694 106.426 180) (fields_autoplaced)
     (effects (font (size 1.27 1.27)) (justify right))
-    (property "Intersheet References" "${INTERSHEET_REFS}" (id 0) (at 210.2333 106.3466 0)
+    (property "Intersheet References" "${INTERSHEET_REFS}" (id 0) (at 211.5033 106.3466 0)
       (effects (font (size 1.27 1.27)) (justify right) hide)
     )
@@
       (effects (font (size 1.524 1.524)))
     )
-    (property "Value" "ProMicro_r" (id 1) (at 231.902 40.64 0)
+    (property "Value" "" (id 1) (at 231.902 40.64 0)
       (effects (font (size 1.524 1.524)))
     )
-    (property "Footprint" "kbd:ProMicro_v3.5" (id 2) (at 229.362 88.9 90)
+    (property "Footprint" "" (id 2) (at 229.362 88.9 90)
       (effects (font (size 1.524 1.524)) hide)
     )
@@
     )
     (path "/2451d668-51ff-44ab-acfe-cfe666fa0c7e"
-      (reference "U1") (unit 1) (value "ProMicro_r") (footprint "kbd:ProMicro_v3.5")
+      (reference "U1") (unit 1) (value "ProMicro_r") (footprint "Alaa:ProMicro2")
     )
     (path "/14d177e6-f355-4bb1-8f3c-ce81903ebacb"
