File: boards/36keys/Batreeq36/Batreeq36.kicad_sch (KiCad schematic)
At the start: 169 parts, among them J1 Conn_01x12_Female, J2 Conn_01x12_Female, J3 Conn_01x08_Female, J4 Conn_01x08_Female, SW1 SW_Push, SW10 SW_Push, SW11 SW_Push, SW12 SW_Push, SW13 SW_Push, SW14 SW_Push, SW15 SW_Push, SW16 SW_Push, SW17 SW_Push, SW18 SW_Push, SW19 SW_Push, SW2 SW_Push, SW20 SW_Push, SW21 SW_Push, SW22 SW_Push, SW23 SW_Push, SW24 SW_Push, SW25 SW_Push, SW26 SW_Push, SW28 SW_Push, SW29 SW_Push, SW3 SW_Push, SW30 SW_Push, SW31 SW_Push, SW32 SW_Push, SW33 SW_Push, SW34 SW_Push, SW35 SW_Push, SW36 RotaryEncoder, SW37 SW_SPDT, SW38 SW_Push, SW39 SW_Push, SW4 SW_Push, SW40 SW_Push, SW41 SW_Push, SW42 SW_Push, SW43 SW_Push, SW44 SW_Push, SW45 SW_Push, SW5 SW_Push, SW6 SW_Push, SW7 SW_Push, SW8 SW_Push, SW9 SW_Push, U1 Elite-C, U2 74HC595, U3 TCR2EF19,LM(CT, U4 PMW3360DM-T2QU, U5 DRV2605L, U6 74LVC1T45

Commit message: batreeq36 not routed yet
Parts:
- removed H6, H7: MountingHole_Pad, Alaa:MountingHole_M3, symbol Mechanical:MountingHole
- added D27, D43: 1N4148, Diode_SMD:D_SOD-123, symbol alaa:Diode_1N4148
- added D41, D92: SK6812MINI-E, Alaa:MX_SK6812MINI-E_REV, symbol kicad-keyboard-parts:SK6812MINI-E
- added SW27, SW46: SW_Push, Alaa:Kailh_hotswap_only_MX-CHOC, symbol Switch:SW_Push
- D90: renamed from D72; value SK6812MINI-E -> (none); footprint Alaa:MX_SK6812MINI-E_REV -> (none)
- renumbered D41 to D42, D83 to D44, D42 to D45, D44 to D46, D45 to D47, D46 to D48, D47 to D49, D84 to D50, D48 to D51, D49 to D52, D50 to D53, D51 to D54, D52 to D55, D53 to D56, D85 to D57, D54 to D58, D55 to D59, D56 to D60, D57 to D61, D58 to D62, D59 to D63, D86 to D64, D60 to D65, D61 to D66, D62 to D67, D63 to D68, D64 to D69, D87 to D70, D88 to D71, D65 to D72, D66 to D73, D67 to D74, D68 to D83, D69 to D84, D74 to D85, D89 to D86, D90 to D87, D70 to D88, D71 to D89, D73 to D91
Connections:
- net GND: now also D41.3 (VSS), D92.3 (VSS)
- net LED_PWR: now also D41.1 (VDD), D92.1 (VDD)
- net col0: now also D6.2 (A)
- net col1: now also D10.2 (A); no longer D6.2 (A)
- net col2: now also D15.2 (A); no longer D10.2 (A)
- net col3: now also D20.2 (A); no longer D15.2 (A)
- net col4: now also D23.2 (A); no longer D20.2 (A)
- net col5: now also D27.2 (A); no longer D23.2 (A)
- net col7: now also D43.2 (A)
- net row_2: now also SW27.1, SW46.1
- net at D87.2 (DOUT): now also D92.4 (DIN)
- net at D52.4 (DIN): now also D41.2 (DOUT); no longer D85.2 (DOUT)
- new net: D27.1 (K), SW27.2
- new net: D41.4 (DIN), D85.2 (DOUT)
- new net: D43.1 (K), SW46.2

Commit message: batreeq 36
Parts:
- removed JP1, JP2, JP3, JP4, JP5, JP6: Jumper_2_Open, Jumper:SolderJumper-2_P1.3mm_Open_TrianglePad1.0x1.5mm, symbol Jumper:Jumper_2_Open
- added JP1: SolderJumper_3_Open, Jumper:SolderJumper-3_P1.3mm_Open_RoundedPad1.0x1.5mm_NumberLabels, symbol Jumper:SolderJumper_3_Open
- D90: value (none) -> SK6812MINI-E; footprint (none) -> Alaa:MX_SK6812MINI-E_REV
- U1: footprint Alaa:Helios-SeaPicro-Nano -> Alaa:Helios-SeaPicro
Connections:
- net LED_3V3: now also U6.3 (A)
- net LED_5V: now also JP1.1 (A)
- net LED_DO: now also JP1.2 (C); no longer U6.4 (B)
- net RAW: now also C6.1, F1.2
- new net LED_SHFT_5V: JP1.3 (B), U6.4 (B)

Commit message: Batreeq36
Parts:
- added J5: Conn_01x03_Female, Connector_PinHeader_2.54mm:PinHeader_1x03_P2.54mm_Vertical, symbol Connector:Conn_01x03_Female
- HAT1: footprint Alaa:5Way-K1-1506DN-01 -> Alaa:5Way-non-reverse
- U6: value 74LVC1T45 -> (none); footprint josh-soic-sot-etc:SOT-563 -> (none); LCSC C352970 -> C139353
Connections:
- net GPIO16: now reaches U1.29 (F0)
- net GPIO16: now also J5.3 (Pin_3)
- net GPIO10: now reaches U1.31 (GPIO10)
- net GPIO10: now also J5.1 (Pin_1)
- net GPIO11: now reaches U1.32 (GPIO11)
- net GPIO11: now also J5.2 (Pin_2)
- no-connect marks 13 -> 12
Changed lines of the file:
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@@
   (no_connect (at 272.288 106.68))
   (no_connect (at 366.014 176.022))
-  (no_connect (at 265.176 78.74))
   (wire (pts (xy 527.685 104.775) (xy 539.115 104.775))
     (stroke (width 0) (type default) (color 0 0 0 0))
@@
     )
   )
+  (global_label "GPIO16" (shape input) (at 239.776 256.286 180) (fields_autoplaced)
+    (effects (font (size 1.27 1.27)) (justify right))
+    (property "Intersheet References" "${INTERSHEET_REFS}" (id 0) (at 230.4686 256.2066 0)
+      (effects (font (size 1.27 1.27)) (justify right) hide)
+    )
+  )
+  (global_label "GPIO11" (shape input) (at 266.446 33.02 90) (fields_autoplaced)
+    (effects (font (size 1.27 1.27)) (justify left))
+    (property "Intersheet References" "${INTERSHEET_REFS}" (id 0) (at 266.3666 23.7126 90)
+      (effects (font (size 1.27 1.27)) (justify left) hide)
+    )
+  )
   (global_label "row_4" (shape input) (at 242.316 66.04 180) (fields_autoplaced)
     (effects (font (size 1.27 1.27)) (justify right))
@@
     )
   )
+  (global_label "GPIO10" (shape input) (at 239.776 251.206 180) (fields_autoplaced)
+    (effects (font (size 1.27 1.27)) (justify right))
+    (property "Intersheet References" "${INTERSHEET_REFS}" (id 0) (at 230.4686 251.1266 0)
+      (effects (font (size 1.27 1.27)) (justify right) hide)
+    )
+  )
   (global_label "SDA" (shape input) (at 242.316 50.8 180) (fields_autoplaced)
     (effects (font (size 1.27 1.27)) (justify right))
@@
     )
   )
+  (global_label "GPIO11" (shape input) (at 239.776 253.746 180) (fields_autoplaced)
+    (effects (font (size 1.27 1.27)) (justify right))
+    (property "Intersheet References" "${INTERSHEET_REFS}" (id 0) (at 230.4686 253.6666 0)
+      (effects (font (size 1.27 1.27)) (justify right) hide)
+    )
+  )
   (global_label "SCLK" (shape input) (at 366.014 155.702 180) (fields_autoplaced)
     (effects (font (size 1.27 1.27)) (justify right))
@@
     )
   )
+  (global_label "GPIO10" (shape input) (at 253.746 33.02 90) (fields_autoplaced)
+    (effects (font (size 1.27 1.27)) (justify left))
+    (property "Intersheet References" "${INTERSHEET_REFS}" (id 0) (at 253.6666 23.7126 90)
+      (effects (font (size 1.27 1.27)) (justify left) hide)
+    )
+  )
   (global_label "col3" (shape output) (at 81.026 238.76 270) (fields_autoplaced)
     (effects (font (size 1.27 1.27)) (justify right))
@@
     )
   )
+  (global_label "GPIO16" (shape input) (at 265.176 78.74 270) (fields_autoplaced)
+    (effects (font (size 1.27 1.27)) (justify right))
+    (property "Intersheet References" "${INTERSHEET_REFS}" (id 0) (at 265.0966 88.0474 90)
+      (effects (font (size 1.27 1.27)) (justify right) hide)
+    )
+  )
   (global_label "LED_3V3" (shape input) (at 277.876 55.88 0) (fields_autoplaced)
     (effects (font (size 1.27 1.27)) (justify left))
@@
     (in_bom yes) (on_board yes)
     (property "Reference" "U6" (id 0) (at 320.167 222.758 0))
-    (property "Value" "74LVC1T45" (id 1) (at 335.407 222.758 0))
-    (property "Footprint" "josh-soic-sot-etc:SOT-563" (id 2) (at 327.152 243.078 0)
+    (property "Value" "" (id 1) (at 335.407 222.758 0))
+    (property "Footprint" "" (id 2) (at 327.152 243.078 0)
       (effects (font (size 1.27 1.27)) hide)
     )
@@
       (effects (font (size 1.27 1.27)) hide)
     )
-    (property "LCSC" "C352970" (id 5) (at 327.152 231.648 0)
+    (property "LCSC" "C139353" (id 5) (at 327.152 231.648 0)
       (effects (font (size 1.27 1.27)) hide)
     )
@@
     (pin "2")
   )
+  (symbol (lib_id "Connector:Conn_01x03_Female") (at 244.856 253.746 0) (unit 1)
+    (in_bom yes) (on_board yes) (fields_autoplaced)
+    (property "Reference" "J5" (id 0) (at 246.38 252.4759 0)
+      (effects (font (size 1.27 1.27)) (justify left))
+    )
+    (property "Value" "Conn_01x03_Female" (id 1) (at 246.38 255.0159 0)
+      (effects (font (size 1.27 1.27)) (justify left))
+    )
+    (property "Footprint" "Connector_PinHeader_2.54mm:PinHeader_1x03_P2.54mm_Vertical" (id 2) (at 244.856 253.746 0)
+      (effects (font (size 1.27 1.27)) hide)
+    )
+    (property "Datasheet" "~" (id 3) (at 244.856 253.746 0)
+      (effects (font (size 1.27 1.27)) hide)
+    )
+    (pin "1")
+    (pin "2")
+    (pin "3")
+  )
   (symbol (lib_id "kicad-keyboard-parts:SK6812MINI-E") (at 512.445 71.12 0) (unit 1)
     (in_bom yes) (on_board yes)
@@
     (property "Reference" "HAT1" (id 0) (at 54.356 213.7918 0))
     (property "Value" "5Way-Tactile_K1-1506DN-01" (id 1) (at 54.356 216.1032 0))
-    (property "Footprint" "Alaa:5Way-K1-1506DN-01" (id 2) (at 38.481 219.075 0)
+    (property "Footprint" "Alaa:5Way-non-reverse" (id 2) (at 38.481 219.075 0)
       (effects (font (size 1.27 1.27)) hide)
     )
@@
     )
     (path "/a79702ed-70ef-421e-beba-55a5423a3e4c"
-      (reference "HAT1") (unit 1) (value "5Way-Tactile_K1-1506DN-01") (footprint "Alaa:5Way-K1-1506DN-01")
+      (reference "HAT1") (unit 1) (value "5Way-Tactile_K1-1506DN-01") (footprint "Alaa:5Way-non-reverse")
     )
     (path "/e3961296-b4c5-459d-a7b6-a37ca9fc9b04"
@@
       (reference "J4") (unit 1) (value "Conn_01x08_Female") (footprint "Alaa:3JST_BAT")
     )
+    (path "/96eaabbc-1351-42a0-b385-94516fb78638"
+      (reference "J5") (unit 1) (value "Conn_01x03_Female") (footprint "Connector_PinHeader_2.54mm:PinHeader_1x03_P2.54mm_Vertical")
+    )
     (path "/7c029c7b-1c91-4623-981d-eb72b148636d"
       (reference "JP1") (unit 1) (value "SolderJumper_3_Open") (footprint "Jumper:SolderJumper-3_P1.3mm_Open_RoundedPad1.0x1.5mm_NumberLabels")
@@
     )
     (path "/2e5fbd59-f8ae-420c-b89e-8c299bbfff35"
-      (reference "U6") (unit 1) (value "74LVC1T45") (footprint "josh-soic-sot-etc:SOT-563")
+      (reference "U6") (unit 1) (value "74LVC1T45") (footprint "Package_TO_SOT_SMD:SOT-363_SC-70-6")
     )
   )
