File: boards/40keys/Zazu/Zazu.kicad_sch (KiCad schematic)
At the start: 175 parts, among them J1 Conn_01x12_Female, J2 Conn_01x12_Female, J3 Conn_01x08_Female, J4 Conn_01x08_Female, J5 Conn_01x03_Female, SW1 SW_Push, SW10 SW_Push, SW11 SW_Push, SW12 SW_Push, SW13 SW_Push, SW14 SW_Push, SW15 SW_Push, SW16 SW_Push, SW17 SW_Push, SW18 SW_Push, SW19 SW_Push, SW2 SW_Push, SW20 SW_Push, SW21 SW_Push, SW22 SW_Push, SW23 SW_Push, SW24 SW_Push, SW25 SW_Push, SW26 SW_Push, SW27 SW_Push, SW28 SW_Push, SW29 SW_Push, SW3 SW_Push, SW30 SW_Push, SW31 SW_Push, SW32 SW_Push, SW33 SW_Push, SW34 SW_Push, SW35 SW_Push, SW36 RotaryEncoder, SW37 SW_SPDT, SW38 SW_Push, SW39 SW_Push, SW4 SW_Push, SW40 SW_Push, SW41 SW_Push, SW42 SW_Push, SW43 SW_Push, SW44 SW_Push, SW45 SW_Push, SW46 SW_Push, SW5 SW_Push, SW6 SW_Push, SW7 SW_Push, SW8 SW_Push, SW9 SW_Push, U1 Elite-C, U2 74HC595, U3 TCR2EF19,LM(CT, U4 PMW3360DM-T2QU, U5 DRV2605L, U6 74LVC1T45

Commit message: zazu fix rgb chain
Changed lines of the file:
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@@
   (junction (at 114.3 87.63) (diameter 0) (color 0 0 0 0)
-  )
-  (junction (at 457.962 145.796) (diameter 0) (color 0 0 0 0)
   )
   (junction (at 450.342 153.416) (diameter 0) (color 0 0 0 0)
@@
     (stroke (width 0) (type default) (color 0 0 0 0))
   )
-  (wire (pts (xy 457.9492 145.7941) (xy 458.978 145.796))
-    (stroke (width 0) (type default) (color 0 0 0 0))
-  )
   (wire (pts (xy 83.82 114.3) (xy 99.06 114.3))
     (stroke (width 0) (type default) (color 0 0 0 0))
@@
     (stroke (width 0) (type default) (color 0 0 0 0))
   )
+  (wire (pts (xy 457.962 145.796) (xy 458.978 145.796))
+    (stroke (width 0) (type default) (color 0 0 0 0))
+  )
