File: boards/30keys/wired-wizza/wired-wizza.kicad_sch (KiCad schematic)
At the start: 176 parts, among them J1 Conn_01x08_Female, J10 Conn_01x08, J2 AudioJack4dpb, J3 Conn_01x12_Female, J4 Conn_01x12_Female, J5 AudioJack4dpb, J6 Conn_01x12_Female, J7 Conn_01x08_Female, J8 Conn_01x12_Female, J9 Conn_01x08, SW1 SW_Push, SW10 SW_Push, SW11 SW_Push, SW12 SW_Push, SW13 SW_Push, SW14 SW_Push, SW15 SW_Push, SW16 SW_Push, SW17 SW_Push, SW18 SW_Push, SW19 SW_Push, SW2 SW_Push, SW20 SW_Push, SW22 SW_Push, SW23 SW_Push, SW24 SW_Push, SW25 SW_Push, SW26 SW_Push, SW27 SW_Push, SW28 SW_Push, SW29 SW_Push, SW3 SW_Push, SW30 SW_Push, SW31 SW_Push, SW32 SW_Push, SW33 SW_Push, SW34 SW_Push, SW35 SW_Push, SW36 Rotary_Encoder_Switch, SW36 SW_Push, SW37 SW_Push, SW38 SW_Push, SW4 SW_Push, SW40 SW_Push, SW5 SW_Push, SW6 SW_Push, SW7 SW_Push, SW8 SW_Push, SW9 SW_Push, U1 Helios, U10 PMW3360DM-T2QU, U2 74LVC1T45, U3 TCR2EF19,LM(CT, U4 PMW3360DM-T2QU, U5 DRV2605L, U6 DRV2605L, U7 Helios, U8 TCR2EF19,LM(CT, U9 74LVC1T45

Commit message: fix wired wizza LEDs
Parts:
- removed U2, U9: 74LVC1T45, Package_TO_SOT_SMD:SOT-363_SC-70-6, symbol Logic_LevelTranslator:SN74LVC1T45DRL
Connections:
- net Backlight is gone; now on an unnamed net: D88.4 (DIN)
- net Backlight_L is gone; now on an unnamed net: D4.4 (DIN)
- net row_4: now also U7.18 (A1/PF6); no longer U7.31 (GPIO10)
- net row_4_L: now also U1.18 (A1/PF6); no longer U1.31 (GPIO10)
- no-connect marks 28 -> 30
Other:
- note removed: "3v3 -> 5V logic shift"
- note removed: "WS2812 Driver"
