File: boards/30keys/Wizza-Choc-VIK/Wizza-Choc-VIK.kicad_pcb (KiCad board)
At the start: 2 copper layers, 214.5 x 80.9 mm, 90 parts, among them J1 AudioJack4dpb, J11 Conn_01x05, J2 AudioJack4dpb, J3 Conn_01x03_Socket, J4 Conn_01x03_Socket, J9 Conn_01x05, SW1 SW_Push, SW10 SW_Push, SW11 SW_Push, SW12 SW_Push, SW13 SW_Push, SW14 SW_Push, SW15 SW_Push, SW16 SW_Push, SW17 SW_Push, SW18 SW_Push, SW19 SW_Push, SW2 SW_Push, SW20 SW_Push, SW21 SW_Push, SW22 SW_Push, SW23 SW_SPDT, SW24 SW_SPDT, SW25 SW_Push, SW26 SW_Push, SW27 SW_Push, SW28 SW_Push, SW29 SW_Push, SW3 SW_Push, SW30 SW_Push, SW31 SW_Push, SW32 SW_Push, SW33 SW_Push, SW34 SW_Push, SW35 Rotary_Encoder_Switch, SW36 Rotary_Encoder_Switch, SW4 SW_Push, SW5 SW_Push, SW6 SW_Push, SW7 SW_Push, SW8 SW_Push, SW9 SW_Push, U3 Helios, U4 Helios

Commit message: wizza vik
Parts:
- moved SW11 210.4 mm to (321.7, 97.6), turned to 90 degrees
- moved SW12 210.2 mm to (111.3, 97.6)
- moved SW1 3.00 mm to (232.1, 72.6)
- moved SW10 3.00 mm to (200.6, 72.6)
- moved SW13 3.00 mm to (232.1, 90.1)
- moved SW14 3.00 mm to (250.6, 81.4)
- moved SW2 3.00 mm to (250.6, 63.9)
- moved SW21 3.00 mm to (182.1, 81.4)
- moved SW22 3.00 mm to (200.6, 90.1)
- moved SW27 3.00 mm to (250.6, 98.9)
- moved SW32 3.00 mm to (182.1, 98.9)
- moved SW9 3.00 mm to (182.1, 63.9)
- moved D28 2.46 mm to (152.4, 100.2)
- moved D12 2.31 mm to (209.2, 74.5)
- moved D11 2.30 mm to (190.7, 65.8)
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Connections:
- J5 pad 11: MOSI_L -> MISO_L
- J6 pad 11: MOSI_R -> MISO_R
- J7 pad 11: MOSI_L -> MISO_L
- J8 pad 11: MOSI_R -> MISO_R
- SW35 pad A: ENC_L_L -> EncR_L
- SW35 pad B: ENC_R_L -> EncL_L
- SW36 pad A: ENC_R_R -> EncR_R
- SW36 pad B: ENC_L_R -> EncL_R
Routing:
- net RAW_L: track 0.00 -> 276.2 mm, vias 0 -> 5
- net row_0_L: track 0.00 -> 216.4 mm, vias 0 -> 11
- net GPIO10_L: track 0.00 -> 197.2 mm, vias 0 -> 4
- net GPIO14_L: track 0.00 -> 186.5 mm, vias 0 -> 2
- net row_1_L: track 0.00 -> 180.1 mm, vias 0 -> 9
- net row_2_L: track 0.00 -> 179.5 mm, vias 0 -> 11
- net GPIO11_L: track 0.00 -> 168.5 mm, vias 0 -> 1
- net GPIO16_L: track 0.00 -> 154.8 mm, vias 0 -> 5
- net GPIO15_L: track 0.00 -> 152.2 mm, vias 0 -> 5
- net col4_L: track 0.00 -> 149.7 mm, vias 0 -> 5
- net TX_L: track 0.00 -> 144.2 mm, vias 0 -> 3
- net col3_L: track 0.00 -> 138.9 mm, vias 0 -> 5
- net RX_L: track 0.00 -> 138.5 mm, vias 0 -> 4
- net SDA_L: track 0.00 -> 133.6 mm, vias 0 -> 4
- net col2_L: track 0.00 -> 129.7 mm, vias 0 -> 6
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- added copper zone on B.Cu, net GND_L
- added copper zone on F.Cu, net GND_L
- added copper zone on B.Cu, net GND_R
- added copper zone on F.Cu, net GND_R

Commit message: wizza vik choc
Parts:
- moved D13 3.30 mm to (240.7, 92.7)
- moved D14 3.23 mm to (259.6, 84.0)
- moved D3 2.00 mm to (240.8, 75.2)
- moved D4 1.29 mm to (259.6, 65.8)
- moved D25 0.54 mm to (259.1, 99.6)
- turned SW11 to -90 degrees
- turned SW36 to 180 degrees
Routing:
- net RAW_R: track 0.00 -> 202.7 mm, vias 0 -> 6
- net GPIO11_R: track 0.00 -> 182.8 mm, vias 0 -> 1
- net row_0_R: track 0.00 -> 170.9 mm, vias 0 -> 8
- net GPIO10_R: track 0.00 -> 163.7 mm, vias 0 -> 4
- net TX_R: track 0.00 -> 158.2 mm, vias 0 -> 3
- net GPIO14_R: track 0.00 -> 152.4 mm, vias 0 -> 2
- net RX_R: track 0.00 -> 144.2 mm, vias 0 -> 2
- net row_2_R: track 0.00 -> 143.5 mm, vias 0 -> 8
- net row_1_R: track 0.00 -> 142.4 mm, vias 0 -> 7
- net GPIO16_R: track 0.00 -> 133.6 mm, vias 0 -> 2
- net GPIO15_R: track 0.00 -> 133.6 mm, vias 0 -> 2
- net col3_R: track 0.00 -> 133.2 mm, vias 0 -> 5
- net col4_R: track 0.00 -> 132.6 mm, vias 0 -> 5
- net VCC_R: track 0.00 -> 125.2 mm, vias 0 -> 6
- net VIK_AD1_R: track 0.00 -> 112.1 mm, vias 0 -> 3
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
Commit message: wizza mx new gerbers
Routing:
- net GND_L: vias 34 -> 35
