File: boards/30keys/Wizza-MX-VIK/Wizza-MX-VIK.kicad_pcb (KiCad board)
At the start: 2 copper layers, 227.5 x 87.4 mm, 90 parts, among them J10 Conn_01x03_Socket, J3 AudioJack4dpb, J4 AudioJack4dpb, J7 Conn_01x05, J8 Conn_01x05, J9 Conn_01x03_Socket, SW1 SW_Push, SW10 SW_Push, SW11 SW_Push, SW12 SW_Push, SW13 SW_Push, SW14 SW_Push, SW15 SW_Push, SW16 SW_Push, SW17 SW_Push, SW18 SW_Push, SW19 SW_Push, SW2 SW_Push, SW20 SW_Push, SW21 SW_Push, SW22 SW_Push, SW23 SW_SPDT, SW24 SW_SPDT, SW25 SW_Push, SW26 SW_Push, SW27 SW_Push, SW28 SW_Push, SW29 SW_Push, SW3 SW_Push, SW30 SW_Push, SW31 SW_Push, SW32 SW_Push, SW33 SW_Push, SW34 SW_Push, SW35 Rotary_Encoder_Switch, SW36 Rotary_Encoder_Switch, SW4 SW_Push, SW5 SW_Push, SW6 SW_Push, SW7 SW_Push, SW8 SW_Push, SW9 SW_Push, U1 Helios, U2 Helios

Commit message: wizza mx vik
Parts:
- removed mouse-bite-2mm-slot (x2): VAL**, Duckyb-Parts:mouse-bite-5mm-slot-with-space-for-track
- moved D27 2.92 mm to (279.3, 124.6)
- turned SW16 to 172 degrees
- turned SW19 to -172 degrees
- turned SW20 to -175 degrees
- turned SW30 to -172 degrees
- turned SW31 to -175 degrees
- turned SW36 to 180 degrees
Connections:
- J1 pad 11: MOSI_R -> MISO_R
- J2 pad 11: MOSI_L -> MISO_L
- J5 pad 11: MOSI_R -> MISO_R
- J6 pad 11: MOSI_L -> MISO_L
- SW35 pad A: ENC_L_L -> EncL_L
- SW35 pad B: ENC_R_L -> EncR_L
- SW36 pad A: ENC_R_R -> EncR_R
- SW36 pad B: ENC_L_R -> EncL_R
Routing:
- net RAW_R: track 0.00 -> 224.9 mm, vias 0 -> 5
- net GPIO14_R: track 0.00 -> 211.2 mm, vias 0 -> 1
- net RAW_L: track 0.00 -> 202.5 mm, vias 0 -> 4
- net GPIO16_L: track 0.00 -> 202.0 mm, vias 0 -> 3
- net GPIO15_L: track 0.00 -> 200.9 mm, vias 0 -> 3
- net GPIO11_R: track 0.00 -> 199.9 mm
- net row_0_L: track 0.00 -> 196.9 mm, vias 0 -> 2
- net GPIO10_L: track 0.00 -> 196.6 mm, vias 0 -> 1
- net row_1_R: track 0.00 -> 194.1 mm, vias 0 -> 10
- net GPIO14_L: track 0.00 -> 193.4 mm, vias 0 -> 1
- net row_0_R: track 0.00 -> 187.8 mm, vias 0 -> 3
- net GPIO15_R: track 0.00 -> 185.5 mm, vias 0 -> 1
- net GPIO11_L: track 0.00 -> 181.4 mm, vias 0 -> 2
- net row_2_L: track 0.00 -> 179.9 mm, vias 0 -> 5
- net GPIO10_R: track 0.00 -> 179.4 mm
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- added copper zone on B.Cu, net GND_L
- added copper zone on F.Cu, net GND_L
- added copper zone on B.Cu, net GND_R
- added copper zone on F.Cu, net GND_R

Commit message: wizza vik
Parts:
- moved D12 3.00 mm to (187.2, 97.2)
- moved D22 3.00 mm to (186.9, 117.0)
- moved SW1 3.00 mm to (228.8, 93.7)
- moved SW10 3.00 mm to (194.8, 93.7)
- moved SW13 3.00 mm to (228.8, 113.2)
- moved SW14 3.00 mm to (248.3, 103.4)
- moved SW2 3.00 mm to (248.3, 83.9)
- moved SW21 3.00 mm to (175.3, 103.4)
- moved SW22 3.00 mm to (194.8, 113.2)
- moved SW27 3.00 mm to (248.3, 122.9)
- moved SW32 3.00 mm to (175.3, 122.9)
- moved SW9 3.00 mm to (175.3, 83.9)
- moved D30 2.31 mm to (165.0, 123.3)
- moved D14 0.50 mm to (240.6, 105.0)
Routing:
- net row_0_L: track 196.9 -> 204.5 mm
- net row_0_R: track 187.8 -> 194.5 mm
- net row_1_L: track 170.1 -> 175.5 mm
- net row_1_R: track 194.1 -> 191.1 mm
- net Net-(D3-K): track 9.12 -> 6.12 mm
- net Net-(D11-K): track 9.84 -> 6.84 mm
- net Net-(D4-K): track 9.96 -> 6.96 mm
- net Net-(D25-K): track 10.4 -> 7.41 mm
- net Net-(D21-K): track 8.76 -> 5.76 mm
- net Net-(D13-K): track 9.64 -> 6.64 mm
- net Net-(D14-K): track 8.92 -> 6.42 mm
- net row_2_L: track 179.9 -> 182.2 mm
- net row_2_R: track 158.5 -> 160.8 mm
- net col2_L: track 128.8 -> 127.6 mm
- net Net-(D30-K): track 8.59 -> 9.62 mm
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
Commit message: add vik 18 pin ffc
Parts:
- added J11: Conn_01x18, Alaa:FPC-SMD_FPC05018-09200-.5mm-rev, B.Cu at (205.9, 101.2)
- added J12: Conn_01x18, Alaa:FPC-SMD_FPC05018-09200-.5mm-rev, B.Cu at (217.9, 101.2)
- added mouse-bite-2mm-slot: VAL**, Duckyb-Parts:mouse-bite-5mm-slot-with-space-for-track, F.Cu at (211.9, 121.6)
- added mouse-bite-2mm-slot: VAL**, Duckyb-Parts:mouse-bite-5mm-slot-with-space-for-track, F.Cu at (211.9, 89.0)
- moved SW23 48.1 mm to (223.7, 152.0), turned to 0 degrees
- moved SW24 45.1 mm to (196.0, 152.0), turned to 0 degrees
- moved D3 4.03 mm to (223.5, 98.3)
Routing:
- net RAW_L: track 202.5 -> 265.9 mm, vias 4 -> 7
- net BAT_L: track 127.5 -> 77.2 mm
- net VCC_L: track 125.2 -> 163.8 mm, vias 3 -> 5
- net SDA_L: track 120.7 -> 158.2 mm, vias 2 -> 4
- net SCL_L: track 121.3 -> 158.2 mm, vias 2 -> 4
- net VCC_R: track 129.1 -> 164.8 mm, vias 1 -> 3
- net SCL_R: track 130.7 -> 165.8 mm, vias 4 -> 6
- net MOSI_R: track 121.7 -> 156.7 mm, vias 3 -> 5
- net SDA_R: track 139.6 -> 174.5 mm, vias 4 -> 6
- net VIK_AD2_R: track 121.1 -> 154.5 mm, vias 1 -> 3
- net NCS_R: track 103.5 -> 136.7 mm, vias 4 -> 6
- net VIK_AD1_R: track 121.4 -> 154.3 mm, vias 3 -> 5
- net MISO_R: track 113.4 -> 143.5 mm, vias 3 -> 5
- net LED_5V_R: track 102.8 -> 132.9 mm, vias 2 -> 4
- net SCLK_R: track 111.1 -> 139.2 mm, vias 2 -> 4
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
Commit message: wizza mx new gerbers
Routing:
- net RAW_R: track 227.0 -> 283.0 mm, vias 5 -> 7
- net GPIO16_L: track 202.0 -> 246.1 mm, vias 3 -> 6
- net GPIO15_L: track 200.9 -> 242.2 mm, vias 3 -> 6
- net MOSI_L: track 103.5 -> 142.7 mm, vias 2 -> 4
- net VIK_AD2_L: track 112.9 -> 152.1 mm, vias 2 -> 4
- net VIK_AD1_L: track 116.4 -> 155.5 mm, vias 2 -> 4
- net GPIO14_L: track 193.4 -> 232.0 mm, vias 1 -> 4
- net LED_5V_L: track 101.1 -> 138.4 mm, vias 1 -> 3
- net GPIO11_L: track 181.4 -> 218.1 mm, vias 2 -> 5
- net GPIO10_L: track 196.6 -> 230.8 mm, vias 1 -> 4
- net NCS_L: track 103.1 -> 136.8 mm, vias 2 -> 4
- net MISO_L: track 100.5 -> 131.3 mm, vias 2 -> 4
- net SCLK_L: track 106.4 -> 136.7 mm, vias 2 -> 4
- net RAW_L: track 265.9 -> 271.4 mm, vias 7 -> 9
- net row_0_L: track 204.5 -> 205.3 mm
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