File: boards/katkoot-vik/Katkoot.kicad_pcb (KiCad board)
At the start: 2 copper layers, 48.9 x 51.2 mm, 16 parts, among them J1 Conn_01x12_Female, J2 Conn_01x12_Female, J3 Conn_01x06_Female, U1 TCR2EF19,LM(CT, U2 PMW3360DM-T2QU

Commit message: VIK Katkoot
Parts:
- removed ? (x2): , 
- removed kibuzzard-63793EB1: G***, kibuzzard-63793EB1
- removed kibuzzard-63793EC8: G***, kibuzzard-63793EC8
- added D1: 1N4148, Diode_SMD:D_SOD-123, B.Cu at (201.2, 65.2)
- added D2: 1N4148, Diode_SMD:D_SOD-123, B.Cu at (201.2, 84.4)
- added D4: 1N4148, Diode_SMD:D_SOD-123, B.Cu at (143.0, 101.1)
- added D5: 1N4148, Diode_SMD:D_SOD-123, B.Cu at (162.1, 101.4)
- added D7: 1N4148, Diode_SMD:D_SOD-123, B.Cu at (181.1, 101.4)
- added D8: 1N4148, Diode_SMD:D_SOD-123, B.Cu at (114.0, 102.3)
- added J4: Conn_01x18, Alaa:FPC-SMD_FPC05018-09200-.5mm-rev, B.Cu at (155.1, 77.9)
- added SW1: Rotary_Encoder_Switch, Alaa:RotaryEncoder_Alps_EC11E-Switch_Vertical_H20mm-keebio_modified, F.Cu at (100.0, 104.9)
- added SW2: SW_Push, Alaa:gateron-ks27-choc-v1-mx-hotswap, F.Cu at (193.7, 69.2)
- added SW3: SW_Push, Alaa:gateron-ks27-choc-v1-mx-hotswap, F.Cu at (193.7, 88.2)
- added SW5: SW_Push, Alaa:gateron-ks27-choc-v1-mx-hotswap, F.Cu at (135.5, 105.7)
- added SW6: SW_Push, Alaa:gateron-ks27-choc-v1-mx-hotswap, F.Cu at (154.5, 105.7)
- added SW8: SW_Push, Alaa:gateron-ks27-choc-v1-mx-hotswap, F.Cu at (173.6, 105.7)
- added U3: xiao-ble, Alaa:xiao-ble-smd-cutout, F.Cu at (192.8, 45.4)
- J1: value Conn_01x12_Female -> ~; footprint Alaa:FPC-SMD_FPC05012-09200-.5mm-rev -> vik:vik-module-connector-horizontal
- J2: value Conn_01x12_Female -> Conn_01x18; footprint Alaa:FPC-SMD_FPC05012-09200-.5mm-rev -> Alaa:FPC-SMD_FPC05018-09200-.5mm-rev
- J3: value Conn_01x06_Female -> Conn_01x18; footprint Connector_PinHeader_2.54mm:PinHeader_1x07_P2.54mm_Vertical -> Alaa:FPC-SMD_FPC05018-09200-.5mm-rev; moved to B.Cu
- moved J2 29.6 mm to (155.3, 90.9), turned to 0 degrees
- moved J1 29.1 mm to (140.4, 58.3), turned to 90 degrees
- moved J3 28.5 mm to (140.7, 72.3)
Connections:
- J1 pad 1: VCC -> SCLK
- J1 pad 10: NCS -> SDA
- J1 pad 11: MISO -> GND
- J1 pad 12: SCLK -> VCC
- J1 pad 2: GND -> MISO
- J1 pad 3: unconnected-(J1-Pad3) -> NCS
- J1 pad 4: unconnected-(J1-Pad4) -> ENC_L
- J1 pad 5: unconnected-(J1-Pad5) -> MOSI
- J1 pad 6: unconnected-(J1-Pad6) -> ENC_R
- J1 pad 7: unconnected-(J1-Pad7) -> RAW
- J1 pad 8: MOSI -> LED_5V
- J1 pad 9: MOTION -> SCL
- J2 pad 1: SCLK -> unconnected-(J2-Pin_1-Pad1)
- J2 pad 10: unconnected-(J2-Pad10) -> ENC_L
- J2 pad 11: GND -> MOSI
- J2 pad 12: VCC -> ENC_R
- J2 pad 13: (no net) -> unconnected-(J2-Pin_13-Pad13)
- J2 pad 14: (no net) -> LED_5V
- J2 pad 2: MISO -> row_0
- J2 pad 3: NCS -> row_1
- J2 pad 4: MOTION -> col0
- J2 pad 5: MOSI -> col1
- J2 pad 6: unconnected-(J2-Pad6) -> col2
- J2 pad 7: unconnected-(J2-Pad7) -> SCLK
- J2 pad 8: unconnected-(J2-Pad8) -> MISO
- J2 pad 9: unconnected-(J2-Pad9) -> NCS
- J3 pad 1: GND -> unconnected-(J3-Pin_1-Pad1)
- J3 pad 2: MISO -> row_0
- J3 pad 3: SCLK -> row_1
- J3 pad 4: MOSI -> col0
- J3 pad 5: NCS -> col1
- J3 pad 6: VCC -> col2
- J3 pad 7: MOTION -> SCLK
- U2 pad 9: MOTION -> unconnected-(U2-MOTION-Pad9)
Routing:
- net NCS: track 112.6 -> 0.00 mm
- net SCLK: track 102.9 -> 0.00 mm
- net VCC: track 88.4 -> 0.00 mm, vias 2 -> 0
- net MOTION: track 80.8 -> 0.00 mm, vias 1 -> 0
- net MISO: track 74.6 -> 0.00 mm
- net MOSI: track 69.3 -> 0.00 mm, vias 1 -> 0
- net VDD: track 51.4 -> 0.00 mm, vias 1 -> 0
- net GND: track 19.6 -> 0.00 mm, vias 6 -> 0
- net Net-(U2-VDDPIX): track 4.76 -> 0.00 mm
- net Net-(U2-~{NRESET}): track 2.40 -> 0.00 mm
- net Net-(U2-LED_P): track 2.03 -> 0.00 mm
Other:
- board size 48.9 x 51.2 mm -> 8.6 x 17.3 mm
