File: boards/30keys/Asfoora - wireless/Asfoora.kicad_pcb (KiCad board)
At the start: 2 copper layers, 245 x 106.5 mm, 78 parts, among them SW10 SW_Push, SW11 SW_Push, SW12 SW_Push, SW13 SW_Push, SW14 SW_Push, SW15 SW_Push, SW17 SW_Push, SW18 SW_Push, SW19 SW_Push, SW2 SW_Push, SW20 SW_Push, SW21 SW_Push, SW22 SW_Push, SW23 SW_Push, SW24 SW_Push, SW25 SW_Push, SW26 SW_Push, SW27 SW_Push, SW28 SW_Push, SW29 SW_Push, SW3 SW_Push, SW30 SW_Push, SW31 SW_Push, SW32 SW_Push, SW33 SW_Push, SW34 SW_SPDT, SW4 SW_Push, SW5 SW_Push, SW6 SW_Push, SW7 SW_Push, SW8 SW_Push, SW9 SW_Push, U1 ProMicro_r

Commit message: fix 5 way switch on wasfoora
Parts:
- turned D15 to 0 degrees
- turned D19 to 0 degrees
- turned D33 to 0 degrees
- turned D34 to 180 degrees
- turned D35 to 180 degrees
Connections:
- D15 pad 1: Net-(D15-K) -> col_0
- D15 pad 2: col_0 -> Net-(D15-A)
- D19 pad 1: Net-(D19-K) -> col_1
- D19 pad 2: col_1 -> Net-(D19-A)
- D33 pad 1: Net-(D33-K) -> col_2
- D33 pad 2: col_2 -> Net-(D33-A)
- D34 pad 1: Net-(D34-K) -> col_3
- D34 pad 2: col_3 -> Net-(D34-A)
- D35 pad 1: Net-(D35-K) -> col_4
- D35 pad 2: col_4 -> Net-(D35-A)
- HAT1 pad 1: Net-(D15-K) -> Net-(D15-A)
- HAT1 pad 2: Net-(D19-K) -> Net-(D19-A)
- HAT1 pad 3: Net-(D33-K) -> Net-(D33-A)
- HAT1 pad 5: Net-(D34-K) -> Net-(D34-A)
- HAT1 pad 6: Net-(D35-K) -> Net-(D35-A)
Routing:
- net Net-(D19-K): track 2.62 -> 0.00 mm
- net Net-(D19-A): track 0.00 -> 2.62 mm
- net Net-(D15-K): track 2.56 -> 0.00 mm
- net Net-(D15-A): track 0.00 -> 2.56 mm
- net Net-(D33-K): track 2.54 -> 0.00 mm
- net Net-(D33-A): track 0.00 -> 2.54 mm
- net Net-(D34-K): track 2.20 -> 0.00 mm
- net Net-(D34-A): track 0.00 -> 2.20 mm
- net Net-(D35-K): track 2.15 -> 0.00 mm
- net Net-(D35-A): track 0.00 -> 2.15 mm
- net bat+: track 30.0 -> 30.6 mm
