File: boards/30keys/Batreeq/Wireless/Batreeq-wireless.kicad_pcb (KiCad board)
At the start: 2 copper layers, 262.4 x 124.1 mm, 107 parts, among them J2 Conn_01x03_Pin, J3 Conn_01x06, SW1 SW_Push, SW10 SW_Push, SW11 SW_Push, SW12 SW_Push, SW13 SW_Push, SW14 SW_Push, SW15 SW_Push, SW16 SW_Push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

Commit message: fix wireless batreeq reset ground pin schematic
Connections:
- SW34 pad 2: gnd -> GND
