File: boards/30keys/Batreeq/Wireless/Batreeq-wireless.kicad_sch (KiCad schematic)
At the start: 105 parts, among them J2 Conn_01x03_Pin, J3 Conn_01x06, SW1 SW_Push, SW10 SW_Push, SW11 SW_Push, SW12 SW_Push, SW13 SW_Push, SW14 SW_Push, SW15 SW_Push, SW16 SW_Push, SW17 SW_Push, SW18 SW_Push, SW19 SW_Push, SW2 SW_Push, SW20 SW_Push, SW21 SW_Push, SW22 SW_Push, SW23 SW_Push, SW24 SW_Push, SW25 SW_SPDT, SW26 SW_Push, SW27 SW_Push, SW28 SW_Push, SW29 SW_Push, SW3 SW_Push, SW30 SW_Push, SW31 SW_Push, SW32 SW_Push, SW33 SW_Push, SW34 SW_Push, SW35 SW_Push, SW37 SW_Push, SW4 SW_Push, SW5 SW_Push, SW6 SW_Push, SW7 SW_Push, SW8 SW_Push, SW9 SW_Push, U4 nice_nano

Commit message: fix wireless batreeq reset ground pin schematic
Connections:
- net gnd is gone; now on net GND: SW34.2
Changed lines of the file:
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@@
     )
   )
-  (global_label "gnd" (shape input) (at 283.21 143.51 0) (fields_autoplaced)
+  (global_label "GND" (shape input) (at 283.21 143.51 0) (fields_autoplaced)
     (effects (font (size 1.27 1.27)) (justify left))
-    (property "Intersheetrefs" "${INTERSHEET_REFS}" (at 288.9305 143.4306 0)
+    (property "Intersheetrefs" "${INTERSHEET_REFS}" (at 289.9863 143.51 0)
       (effects (font (size 1.27 1.27)) (justify left) hide)
     )
